File: Hardware/VehicleControlUnit/Motor_Comms.kicad_sch (KiCad schematic)
At the start: 31 parts, among them IC4 ISO1042QDWRQ1, IC5 ISO7741DWR, IC6 ISO7741DWR, J11 Debug_PinHeader, Q3 IRLML2030TRPBF, Q4 IRLML2030TRPBF, U5 MCP4822

Commit message: mikas paradise
Parts:
- removed C41: 10uF, Capacitor_SMD:C_0603_1608Metric_Pad1.08x0.95mm_HandSolder, symbol Device:C
- removed C42, C43: 2.2uF, Capacitor_SMD:C_0603_1608Metric_Pad1.08x0.95mm_HandSolder, symbol Device:C
- removed J11: Debug_PinHeader, Connector_PinHeader_1.00mm:PinHeader_2x11_P1.00mm_Vertical, symbol Connector_Generic:Conn_02x11_Counter_Clockwise
- removed JP5: SolderJumper_2_Open, Jumper:SolderJumper-2_P1.3mm_Open_RoundedPad1.0x1.5mm, symbol Jumper:SolderJumper_2_Open
- removed L2: 10u, 10uH_inducto:WE-MAIA_2512, symbol Device:L
- removed PS1: ROE-3.305S, ROE-3.305S:CONV_ROE-3.305S, symbol ROE-3.305S:ROE-3.305S
- removed U5: MCP4822, MCP4822T-E_SN:MCP4822T-E_SN, symbol Analog_DAC:MCP4822
- added D? (x4): LED, LED_SMD:LED_0603_1608Metric, symbol Device:LED
- added IC?: ISO7741DWR, ISO7741DWR:ISO7741DWR, symbol ISO7741DWR:ISO7741DWR
- added Q? (x4): IRLML2030TRPBF, IRLML2030TRPBF:IRLML2030TRPBF, symbol Simulation_SPICE:NMOS
- added R? (x6): 10k, Resistor_SMD:R_0603_1608Metric_Pad0.98x0.95mm_HandSolder, symbol Device:R
- added R? (x4): 1k, Resistor_SMD:R_0603_1608Metric_Pad0.98x0.95mm_HandSolder, symbol Device:R
- added TP? (x29): TestPoint, TestPoint:TestPoint_Loop_D2.50mm_Drill1.0mm_LowProfile, symbol Connector:TestPoint
- added U?: MCP4922, symbol Analog_DAC:MCP4922
- R47: value R -> 1k
Connections:
- net F/R_MODE_IN is gone; now on net F/R_MODE_OUT: Q4.1 (D)
- net PWR_MODE_IN is gone; now on net +5V_Mtr: Q3.1 (D)
- net +3.3V: now also IC?.1 (VCC1), R?.1, TP?.1
- net Accel_DAC: now also R?.2, TP?.1, U?.14 (VA)
- net Brake_DAC: now also R?.2, TP?.1, U?.10 (VB)
- net CAN_RX: now also TP?.1
- net CAN_TX: now also TP?.1
- net DAC_CLK: now also TP?.1
- net DAC_CS: now also TP?.1
- net DAC_MOSI: now also TP?.1
- net FWD_EN: now also IC?.4 (INB), TP?.1; no longer IC5.4 (INB)
- net F/R_MODE_OUT: no longer Q4.3 (S)
- net F/R_Mode: now also TP?.1
- net F/R_Mode_Gate: now also IC?.13 (OUTB); no longer IC5.13 (OUTB)
- net GND: now also IC?.2 (GND1_1), IC?.8 (GND1_2), TP?.1; no longer D17.1 (K), D18.1 (K), R50.2
- net GND_ISO: now also D17.1 (K), D18.1 (K), Q4.3 (S), R50.2, D?.1 (K), D?.1 (K), D?.1 (K), D?.1 (K), IC?.15 (GND2_2), IC?.9 (GND2_1), Q?.3 (S), Q?.3 (S), Q?.3 (S), Q?.3 (S), R?.1, R?.1, TP?.1, U?.12 (Vss)
- net LDAC: now also TP?.1
- net Mtr_CANH: now also TP?.1
- net Mtr_CANL: now also TP?.1
- net PWR_MODE_EN: now also IC?.3 (INA), TP?.1; no longer IC5.3 (INA)
- net PwrMode_Gate: now also IC?.14 (OUTA), TP?.1; no longer IC5.14 (OUTA)
- net SPI_CLK_ISO: now also TP?.1, U?.4 (SCK)
- net SPI_CS_ISO: now also R?.1, TP?.1, U?.3 (~{CS})
- net SPI_MOSI_ISO: now also TP?.1, U?.5 (SDI)
- net at JP3.2 (B), JP4.2 (B): now also U?.8 (~{LDAC})
- net Map_Bit3_Gate: now reaches IC5.12 (OUTC)
- net Map_Bit3_Gate: now also Q?.2 (G), R?.2, TP?.1
- net Map_Bit3_G: now reaches IC5.5 (INC)
- net Map_Bit3_G: now also TP?.1
- net +3.3V_ISO renamed +5V_Mtr
- net +5V_Mtr: now also IC?.16 (VCC), R?.1, R?.2, R?.2, TP?.1, U?.1 (Vdd), U?.11 (VrefB), U?.13 (VrefA)
- net Pulse_ADC renamed Pulse_ADC_DIV
- net Pulse_ADC_DIV: now also IC?.11 (IND)
- new net: D?.2 (A), R?.1 (x4)
- new net: IC?.10 (EN2), R?.2
- new net: IC?.7 (EN1), R?.2
- new net: R?.1, U?.9 (~{SHDN})
- new net Map_Bit0_G: IC?.5 (INC), TP?.1
- new net Map_Bit0_Gate: IC?.12 (OUTC), Q?.2 (G), R?.2, TP?.1
- new net Map_Bit0_Sig: Q?.1 (D)
- new net Map_Bit1_G: IC5.3 (INA), TP?.1
- new net Map_Bit1_Gate: IC5.14 (OUTA), Q?.2 (G), R?.2, TP?.1
- new net Map_Bit1_Sig: Q?.1 (D)
- new net Map_Bit2_G: IC5.4 (INB), TP?.1
- new net Map_Bit2_Gate: IC5.13 (OUTB), Q?.2 (G), R?.2, TP?.1
- new net Map_Bit2_Sig: Q?.1 (D)
- new net Map_Bit3_Sig: Q?.1 (D)
- new net Pulse_ADC_ISO: IC?.6 (OUTD)
- no-connect marks 11 -> 8
Other:
- note added: "MAP_GND - Terminal 11"
- note added: "Map Bit Level Shifting"
- note added: "Set GA Bit -> 1, for 0-4.8V"
- note added: "Tereminal 25"
- note added: "Tereminal 5"
- note added: "Tereminal 6"
- note added: "Tereminal 7"
- note added: "Terminal 12"
- note added: "Terminal 13"
- note added: "Terminal 31"
- note added: "Terminal 32"
- note added: "Vth = =1.3V Vgate (max) ~= 3.3V"
- note added: "post: rev a maybe, dac alrady has buffers built in"
- note added: "unity gain buffer for dac? dac -> op amp buff -> output"
- note removed: "Isolated DC-DC"
- note removed: "Tereminal 25/7"
- note removed: "Tereminal 5/6"
- moved on the sheet: C40, C44, C45, D17, D18, IC4, IC5, IC6, JP2, JP3, JP4, Q3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

Commit message: i hate this moco, its so stupid why are we doign this.
Parts:
- removed Q3: IRLML2030TRPBF, IRLML2030TRPBF:IRLML2030TRPBF, symbol Simulation_SPICE:NMOS
- added C44: 4.7uF, symbol Device:C
- added C45, C46: 330pF, symbol Device:C
- added D25: LED, symbol Device:LED
- added JP5: SolderJumper_2_Open, Jumper:SolderJumper-2_P1.3mm_Open_RoundedPad1.0x1.5mm, symbol Jumper:SolderJumper_2_Open
- added L2: 10uH, 10uH_inducto:WE-MAIA_2512, symbol Device:L
- added PS1: ROE-3.305S, ROE-3.305S:CONV_ROE-3.305S, symbol ROE-3.305S:ROE-3.305S
- added Q3: DMP3099L-7, DMP3099L-7:DMP3099L-7, symbol Simulation_SPICE:PMOS
- added R60: 5k, Resistor_SMD:R_0603_1608Metric_Pad0.98x0.95mm_HandSolder, symbol Device:R
- gave numbers to parts that had none: 49
- renumbered C40 to C41, C44 to C42, C45 to C43, D17 to D19, D18 to D20, IC4 to IC7, JP3 to JP2, JP4 to JP3, JP2 to JP4, R41 to R43, R42 to R44, R47 to R45, R48 to R46, R45 to R48, R46 to R49, R43 to R52, R44 to R57, R49 to R61, R50 to R62
Connections:
- net +3.3V: now also JP5.1 (A), L2.1
- net F/R_MODE_OUT: now also Q4.3 (S); no longer Q4.1 (D)
- net GND: now also C44.2, C46.2, PS1.1 (-VIN)
- net GND_ISO: now also C46.1, D25.1 (K), PS1.3 (-VOUT); no longer Q4.3 (S)
- net PWR_MODE_OUT: now also Q3.1 (D)
- net PwrMode_Gate: now also Q3.2 (G)
- net +5V_Mtr renamed +5V_ISO
- net +5V_ISO: now also C45.1, PS1.4 (+VOUT), R60.1; no longer U5.11 (VrefB), U5.13 (VrefA)
- new net: C44.1, C45.2, JP5.2 (B), L2.2, PS1.2 (+VIN)
- new net Accel_Vref: U5.13 (VrefA)
- new net Brake_Vref: U5.11 (VrefB)
- new net F/R_MODE_IN: Q4.1 (D)
- new net LED+: D25.2 (A), R60.2
- new net PWR_MODE_IN: Q3.3 (S)
Other:
- note added: "Isolated 3.3V -> 5V"
- note added: "MoCo LED"
- note added: "Vth = = -1V Negative Logic"
- moved on the sheet: TP10, TP11, TP12, TP13, TP14, TP15, TP16, TP17, TP18, TP19, TP20, TP21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

Commit message: put puzzle togaehtrwetr
Parts:
- added C47: 100nF, Capacitor_SMD:C_0603_1608Metric_Pad1.08x0.95mm_HandSolder, symbol Device:C
- added C48: 4.7uF, Capacitor_SMD:C_0603_1608Metric_Pad1.08x0.95mm_HandSolder, symbol Device:C
- C44, C45, C46: footprint (none) -> Capacitor_SMD:C_0603_1608Metric_Pad1.08x0.95mm_HandSolder
- D25: value LED -> LTST-C193KFKT-5A; footprint (none) -> LED_SMD:LED_0603_1608Metric; now fitted
- U5: value MCP4922 -> MCP4922T-E/ST; footprint (none) -> MCP4922T-EST:MCP4922T-EST
Connections:
- net +5V_ISO: now also C47.1, C48.1; no longer R60.1
- net DAC_CLK: now also IC6.4 (INB); no longer IC6.3 (INA)
- net DAC_CS: now also IC6.3 (INA); no longer IC6.5 (INC)
- net DAC_MOSI: now also IC6.5 (INC); no longer IC6.4 (INB)
- net GND_ISO: now also C47.2, C48.2; no longer D25.1 (K)
- net LED+: now also R60.1; no longer D25.2 (A), R60.2
- net SPI_CLK_ISO: now also IC6.13 (OUTB); no longer IC6.14 (OUTA)
- net SPI_CS_ISO: now also IC6.14 (OUTA); no longer IC6.12 (OUTC)
- net SPI_MOSI_ISO: now also IC6.12 (OUTC); no longer IC6.13 (OUTB)
- net +3.3V_in: now reaches C44.1, C45.2, JP5.2 (B), L2.2, PS1.2 (+VIN)
- new net: D25.2 (A), R60.2
- new net LED-: D25.1 (K)
Other:
- moved on the sheet: C44, C45, C46, JP5, L2, PS1, R60
