File: Hardware/VehicleControlUnit/Motor_Comms.kicad_sch (KiCad schematic)
At the start: 82 parts, among them IC4 ISO7741DWR, IC5 ISO7741DWR, IC6 ISO7741DWR, IC7 ISO1042QDWRQ1, Q3 DMP3099L-7, Q4 IRLML2030TRPBF, Q5 IRLML2030TRPBF, Q6 IRLML2030TRPBF, Q7 IRLML2030TRPBF, Q8 IRLML2030TRPBF, U5 MCP4922T-E/ST

Commit message: layoutttttttttttttttttttttttttttttttttttt
Parts:
- removed TP10, TP11, TP12, TP13, TP14, TP15, TP16, TP17, TP18, TP19, TP20, TP21, TP22, TP23, TP24, TP25, TP26, TP27, TP28, TP29, TP30, TP31, TP32, TP33, TP34, TP35, TP36, TP37, TP38: TestPoint, TestPoint:TestPoint_Loop_D2.50mm_Drill1.0mm_LowProfile, symbol Connector:TestPoint
- added J13: Debug_Conn, Connector_PinHeader_2.54mm:PinHeader_2x15_P2.54mm_Vertical, symbol Connector_Generic:Conn_02x15_Counter_Clockwise
- renumbered D20 to D24, D19 to D25, D21 to D26, D22 to D27, D23 to D28, D24 to D29, D25 to D30, Q4 to Q3, Q3 to Q4, R42 to R47, R43 to R48, R44 to R49, R46 to R50, R45 to R51, R47 to R52, R48 to R53, R49 to R54, R50 to R55, R51 to R56, R52 to R57, R53 to R58, R54 to R59, R55 to R60, R56 to R61, R57 to R62, R58 to R63, R59 to R64, R60 to R65, R61 to R66, R62 to R67
Connections:
- net +3.3V: now also J13.1 (Pin_1)
- net +5V_ISO: now also J13.30 (Pin_30)
- net Accel_DAC: now also J13.4 (Pin_4)
- net Brake_DAC: now also J13.3 (Pin_3)
- net CAN_RX: now also J13.8 (Pin_8)
- net CAN_TX: now also J13.9 (Pin_9)
- net DAC_CLK: now also J13.15 (Pin_15)
- net DAC_CS: now also J13.17 (Pin_17)
- net DAC_MOSI: now also J13.14 (Pin_14)
- net FWD_EN: now also J13.6 (Pin_6)
- net F/R_Mode_Gate: now also J13.27 (Pin_27)
- net GND: now also J13.16 (Pin_16), J13.2 (Pin_2)
- net GND_ISO: now also J13.29 (Pin_29)
- net LDAC: now also J13.5 (Pin_5)
- net Map_Bit0_G: now also J13.10 (Pin_10)
- net Map_Bit0_Gate: now also J13.23 (Pin_23)
- net Map_Bit1_G: now also J13.11 (Pin_11)
- net Map_Bit1_Gate: now also J13.22 (Pin_22)
- net Map_Bit2_G: now also J13.12 (Pin_12)
- net Map_Bit2_Gate: now also J13.21 (Pin_21)
- net Map_Bit3_G: now also J13.13 (Pin_13)
- net Map_Bit3_Gate: now also J13.20 (Pin_20)
- net Mtr_CANH: now also J13.19 (Pin_19)
- net Mtr_CANL: now also J13.18 (Pin_18)
- net PWR_MODE_EN: now also J13.7 (Pin_7)
- net PwrMode_Gate: now also J13.28 (Pin_28)
- net SPI_CLK_ISO: now also J13.24 (Pin_24)
- net SPI_CS_ISO: now also J13.25 (Pin_25)
- net SPI_MOSI_ISO: now also J13.26 (Pin_26)
Other:
- note added: "PwrMode_Gate = 1 || Power mode enabled else Eco mode enabled"
- moved on the sheet: D25, IC5, Q4, R48, R51, R53

Commit message: migtve finally lcokeefd in = ggs
Parts:
- removed J13: Debug_Conn, Connector_PinHeader_2.54mm:PinHeader_2x15_P2.54mm_Vertical, symbol Connector_Generic:Conn_02x15_Counter_Clockwise
- added J14: Debug_Conn1, Connector_PinHeader_2.54mm:PinHeader_2x08_P2.54mm_Vertical, symbol Connector_Generic:Conn_02x08_Counter_Clockwise
- added J15: Debug_Conn2, Connector_PinHeader_2.54mm:PinHeader_2x06_P2.54mm_Vertical, symbol Connector_Generic:Conn_02x06_Counter_Clockwise
- PS1: value ROE-3.305S -> ROE-3.505S; MP ROE-3.305S -> ROE-3.505S
Connections:
- net +3.3V: now also J14.1 (Pin_1); no longer JP5.1 (A), L2.1
- net +5V_ISO: now also J15.1 (Pin_1)
- net Accel_DAC: now also J14.3 (Pin_3)
- net Brake_DAC: now also J14.2 (Pin_2)
- net CAN_RX: now also J14.7 (Pin_7)
- net CAN_TX: now also J14.8 (Pin_8)
- net DAC_CLK: now also J14.10 (Pin_10)
- net DAC_CS: now also J14.9 (Pin_9)
- net DAC_MOSI: now also J14.11 (Pin_11)
- net FWD_EN: now also J14.5 (Pin_5)
- net F/R_Mode_Gate: now also J15.3 (Pin_3)
- net GND: now also J14.16 (Pin_16)
- net GND_ISO: now also J15.12 (Pin_12), J15.7 (Pin_7)
- net LDAC: now also J14.4 (Pin_4)
- net Map_Bit0_G: now also J14.15 (Pin_15)
- net Map_Bit0_Gate: now also J15.11 (Pin_11)
- net Map_Bit1_G: now also J14.14 (Pin_14)
- net Map_Bit1_Gate: now also J15.10 (Pin_10)
- net Map_Bit2_G: now also J14.13 (Pin_13)
- net Map_Bit2_Gate: now also J15.9 (Pin_9)
- net Map_Bit3_G: now also J14.12 (Pin_12)
- net Map_Bit3_Gate: now also J15.8 (Pin_8)
- net PWR_MODE_EN: now also J14.6 (Pin_6)
- net PwrMode_Gate: now also J15.2 (Pin_2)
- net SPI_CLK_ISO: now also J15.6 (Pin_6)
- net SPI_CS_ISO: now also J15.5 (Pin_5)
- net SPI_MOSI_ISO: now also J15.4 (Pin_4)
- net +3.3V_in renamed +5V_in
- new net +5V: JP5.1 (A), L2.1
Other:
- note removed: "Pin Header will be finalized at layout"
- note removed: "post: rev a maybe, dac alrady has buffers built in"
- note removed: "unity gain buffer for dac? dac -> op amp buff -> output"

Commit message: tracing in progress....
Parts:
- added C41, C42, C43, C44, C45, C46, C47, C48, C49, C50, C51, C52, C56, C57, C58, C59: 0.1u, Capacitor_SMD:C_0603_1608Metric_Pad1.08x0.95mm_HandSolder, symbol Device:C
- renumbered C42 to C53, C43 to C54, C41 to C55, C44 to C60, C45 to C61, C46 to C62, C47 to C63, C48 to C64
Connections:
- net +3.3V: now also C41.1, C42.1, C43.1, C44.1, C49.1, C50.1, C56.1, C57.1, C58.1, C59.1
- net +5V_ISO: now also C45.1, C46.1, C47.1, C48.1, C51.1, C52.1
- net GND: now also C41.2, C42.2, C43.2, C44.2, C49.2, C50.2, C56.2, C57.2, C58.2, C59.2
- net GND_ISO: now also C45.2, C46.2, C47.2, C48.2, C51.2, C52.2
Other:
- moved on the sheet: C53, C54, C55, D24, D25, D26, D27, D28, D29, IC4, IC5, IC7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
