File: Hardware/VehicleControlUnit/Motor_Comms.kicad_sch (KiCad schematic)
At the start: 71 parts, among them IC4 ISO7741DWR, IC5 ISO7741DWR, IC6 ISO7741DWR, IC7 ISO1042QDWRQ1, J14 Debug_Conn1, J15 Debug_Conn2, Q3 IRLML2030TRPBF, Q4 DMP3099L-7, Q5 IRLML2030TRPBF, Q6 IRLML2030TRPBF, Q7 IRLML2030TRPBF, Q8 IRLML2030TRPBF, U5 MCP4922T-E/ST

Commit message: 70% tracing done
Parts:
- removed C42, C43, C46, C47, C52, C56, C57, C58, C59: 0.1u, Capacitor_SMD:C_0603_1608Metric_Pad1.08x0.95mm_HandSolder, symbol Device:C
- removed J14: Debug_Conn1, Connector_PinHeader_2.54mm:PinHeader_2x08_P2.54mm_Vertical, symbol Connector_Generic:Conn_02x08_Counter_Clockwise
- removed J15: Debug_Conn2, Connector_PinHeader_2.54mm:PinHeader_2x06_P2.54mm_Vertical, symbol Connector_Generic:Conn_02x06_Counter_Clockwise
- removed JP3, JP4: SolderJumper_2_Bridged, Jumper:SolderJumper-2_P1.3mm_Bridged2Bar_RoundedPad1.0x1.5mm, symbol Jumper:SolderJumper_2_Bridged
- added C51: 0.1u, Capacitor_SMD:C_0603_1608Metric_Pad1.08x0.95mm_HandSolder, symbol Device:C
- added J14: Debug_Conn1, Connector_PinHeader_2.54mm:PinHeader_2x07_P2.54mm_Vertical, symbol Connector_Generic:Conn_02x07_Counter_Clockwise
- added J15: Debug_Conn2, Connector_PinHeader_2.54mm:PinHeader_2x07_P2.54mm_Vertical, symbol Connector_Generic:Conn_02x07_Counter_Clockwise
- added JP3, JP4: SolderJumper_2_Open, Jumper:SolderJumper-2_P1.3mm_Open_RoundedPad1.0x1.5mm, symbol Jumper:SolderJumper_2_Open
- renumbered C44 to C42, C45 to C43, C48 to C44, C49 to C45, C51 to C46, C53 to C47, C54 to C48, C55 to C49, C60 to C52, C61 to C53, C62 to C54, C63 to C55, C64 to C56, R47 to R48, R48 to R49, R49 to R50, R50 to R51, R51 to R52, R52 to R53, R53 to R54, R54 to R55, R55 to R56, R56 to R57, R57 to R58, R58 to R59, R59 to R60, R60 to R61, R61 to R62, R62 to R63, R63 to R65, R65 to R66, R66 to R67, R67 to R68
Connections:
- net +3.3V: now also J14.1 (Pin_1)
- net +5V_ISO: now also C51.1, J15.1 (Pin_1)
- net Accel_DAC: now also J15.14 (Pin_14)
- net Brake_DAC: now also J15.13 (Pin_13)
- net CAN_RX: now also J14.5 (Pin_5)
- net CAN_TX: now also J14.6 (Pin_6)
- net DAC_CLK: now also J14.7 (Pin_7)
- net DAC_CS: now also J14.8 (Pin_8)
- net DAC_MOSI: now also J14.9 (Pin_9)
- net FWD_EN: now also J14.3 (Pin_3)
- net F/R_Mode_Gate: now also J15.4 (Pin_4)
- net GND: now also J14.14 (Pin_14), JP3.1 (A)
- net GND_ISO: now also C51.2, J15.11 (Pin_11), J15.9 (Pin_9)
- net LDAC: now also J14.2 (Pin_2)
- net Map_Bit0_G: now also J14.13 (Pin_13)
- net Map_Bit0_Gate: now also J15.3 (Pin_3)
- net Map_Bit1_G: now also IC4.6 (OUTD), J14.12 (Pin_12); no longer IC5.3 (INA)
- net Map_Bit1_Gate: now also IC4.11 (IND), J15.6 (Pin_6); no longer IC5.14 (OUTA)
- net Map_Bit2_G: now also IC5.3 (INA), J14.11 (Pin_11); no longer IC5.4 (INB)
- net Map_Bit2_Gate: now also IC5.14 (OUTA), J15.5 (Pin_5); no longer IC5.13 (OUTB)
- net Map_Bit3_G: now also IC5.4 (INB), J14.10 (Pin_10); no longer IC5.5 (INC)
- net Map_Bit3_Gate: now also IC5.13 (OUTB), J15.8 (Pin_8); no longer IC5.12 (OUTC)
- net PWR_MODE_EN: now also J14.4 (Pin_4)
- net Pulse_ADC_DIV: now also IC5.12 (OUTC); no longer IC4.11 (IND)
- net Pulse_ADC_ISO: now also IC5.5 (INC); no longer IC4.6 (OUTD)
- net PwrMode_Gate: now also J15.2 (Pin_2)
- net SPI_CLK_ISO: now also J15.10 (Pin_10)
- net SPI_CS_ISO: now also J15.12 (Pin_12)
- net SPI_MOSI_ISO: now also J15.7 (Pin_7)
- net at C49.1, R63.1: now also JP4.2 (B)
- net at R58.2: now also JP4.1 (A)
- net at JP2.2 (B), U5.8 (~{LDAC}): now also JP3.2 (B)
Other:
- note added: "SOLDER"
- moved on the sheet: C41, C42, C43, C44, C45, C46, R64, R65

Commit message: DONEEE - silkscreen time
Parts:
- removed J14: Debug_Conn1, Connector_PinHeader_2.54mm:PinHeader_2x07_P2.54mm_Vertical, symbol Connector_Generic:Conn_02x07_Counter_Clockwise
- added J14: PH1, Connector_PinHeader_2.54mm:PinHeader_1x04_P2.54mm_Vertical, symbol Connector_Generic:Conn_01x04
- added J15: PH2, Connector_PinHeader_2.54mm:PinHeader_1x03_P2.54mm_Vertical, symbol Connector_Generic:Conn_01x03
- added J17: PH4, Connector_PinHeader_2.54mm:PinHeader_1x04_P2.54mm_Vertical, symbol Connector_Generic:Conn_01x04
- added J18: PH3, Connector_PinHeader_2.54mm:PinHeader_1x03_P2.54mm_Vertical, symbol Connector_Generic:Conn_01x03
- renumbered C41 to C42, C42 to C43, C43 to C44, C44 to C45, C45 to C46, C46 to C47, C47 to C48, C48 to C49, C49 to C50, C50 to C51, C51 to C52, C52 to C53, C53 to C54, C54 to C55, C55 to C56, C56 to C57, J15 to J16, R48 to R49, R49 to R50, R50 to R51, R51 to R52, R52 to R53, R53 to R54, R54 to R55, R55 to R56, R56 to R57, R57 to R58, R58 to R59, R59 to R60, R60 to R61, R61 to R62, R62 to R63, R63 to R64, R64 to R65, R65 to R66, R66 to R67, R67 to R68, R68 to R69
Connections:
- net +3.3V: now also J17.1 (Pin_1)
- net CAN_RX: now also J17.2 (Pin_2)
- net CAN_TX: now also J17.3 (Pin_3)
- net DAC_CLK: now also J18.2 (Pin_2)
- net DAC_CS: now also J18.3 (Pin_3)
- net DAC_MOSI: now also J18.1 (Pin_1)
- net FWD_EN: now also J14.2 (Pin_2)
- net GND: now also J17.4 (Pin_4)
- net LDAC: now also J15.2 (Pin_2)
- net Map_Bit0_G: now also J14.3 (Pin_3)
- net Map_Bit1_G: now also J14.4 (Pin_4)
- net Map_Bit2_G: now also J15.1 (Pin_1)
- net Map_Bit3_G: now also J15.3 (Pin_3)
- net PWR_MODE_EN: now also J14.1 (Pin_1)
Other:
- moved on the sheet: J16

Commit message: VCU hardware prod files done night night
Parts:
- renumbered J14 to J15, J15 to J16, J16 to J17, J17 to J18, J18 to J19
Changed lines of the file:
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@@
 		(in_pos_files yes)
 		(dnp no)
-		(property "Reference" "J18"
+		(property "Reference" "J19"
 			(at 207.01 123.19 0)
 			(show_name no)
@@
 			(project "VehicleControlUnit"
 				(path "/e864fac9-3897-46c9-9101-6d5488c6cd3a/351a8545-bbe6-4531-b2a7-55d4b724255d"
-					(reference "J18")
+					(reference "J19")
 					(unit 1)
 				)
@@
 		(in_pos_files yes)
 		(dnp no)
-		(property "Reference" "J15"
+		(property "Reference" "J16"
 			(at 202.946 133.604 0)
 			(show_name no)
@@
 			(project "VehicleControlUnit"
 				(path "/e864fac9-3897-46c9-9101-6d5488c6cd3a/351a8545-bbe6-4531-b2a7-55d4b724255d"
-					(reference "J15")
+					(reference "J16")
 					(unit 1)
 				)
@@
 		(dnp no)
 		(fields_autoplaced yes)
-		(property "Reference" "J16"
+		(property "Reference" "J17"
 			(at 204.724 138.303 0)
 			(show_name no)
@@
 			(project "VehicleControlUnit"
 				(path "/e864fac9-3897-46c9-9101-6d5488c6cd3a/351a8545-bbe6-4531-b2a7-55d4b724255d"
-					(reference "J16")
+					(reference "J17")
 					(unit 1)
 				)
@@
 		(in_pos_files yes)
 		(dnp no)
-		(property "Reference" "J14"
+		(property "Reference" "J15"
 			(at 200.914 106.68 0)
 			(show_name no)
@@
 			(project "VehicleControlUnit"
 				(path "/e864fac9-3897-46c9-9101-6d5488c6cd3a/351a8545-bbe6-4531-b2a7-55d4b724255d"
-					(reference "J14")
+					(reference "J15")
 					(unit 1)
 				)
@@
 		(in_pos_files yes)
 		(dnp no)
-		(property "Reference" "J17"
+		(property "Reference" "J18"
 			(at 209.296 119.634 0)
 			(show_name no)
@@
 			(project "VehicleControlUnit"
 				(path "/e864fac9-3897-46c9-9101-6d5488c6cd3a/351a8545-bbe6-4531-b2a7-55d4b724255d"
-					(reference "J17")
+					(reference "J18")
 					(unit 1)
 				)
