File: Hardware/VehicleControlUnit/VehicleControlUnit.kicad_pcb (KiCad board)
At the start: 4 copper layers, 90 x 60 mm, 178 parts, among them IC1 LM74502DDFR, IC2 TCAN3413DR, IC3 EMC2305-1-AP-TR, IC4 ISO1042QDWRQ1, IC5 ISO7741DWR, IC6 ISO7741DWR, J1 CAN_DEBUG_NANO_01x04, J10 Micro_SD_Card_Det2, J11 Debug_PinHeader, J12 USB_C_Receptacle_USB2.0_16P, J2 CAN_NANO_01x03, J3 CAN_NANO_01x03, J4 Fan_Conn1, J5 Motor_Conn1, J6 Motor_Conn2, J7 Fan_Conn2, J8 SWD_Header, J9 SWD, Q1 PSMN012-100YS, Q2 PSMN012-100YS, Q3 IRLML2030TRPBF, Q4 IRLML2030TRPBF, SW1 SW_SPDT, U1 LMR51635XDDCR, U2 TPS2117DRLR, U3 MCP1826S, U4 STM32G473VETx, U5 MCP4822, Y1 Crystal

Commit message: put puzzle togaehtrwetr
Parts:
- removed the J11 at (121.8, -0.96)
- removed the J12 at (-22.5, 18.9)
- removed the J6 at (166.5, 142.1)
- removed the R15 at (-88.3, 87.4)
- removed the R2 at (71.3, 131.3)
- removed the R34 at (-70.8, 45.3)
- added C47: 100nF, Capacitor_SMD:C_0603_1608Metric_Pad1.08x0.95mm_HandSolder, B.Cu at (134.3, 60.2)
- added C48: 4.7uF, Capacitor_SMD:C_0603_1608Metric_Pad1.08x0.95mm_HandSolder, B.Cu at (131.0, 59.3)
- added C49: 10uF, Capacitor_SMD:C_0805_2012Metric, F.Cu at (180.9, 115.6)
- added D19: LED, LED_SMD:LED_0603_1608Metric, F.Cu at (127.9, 158.1)
- added D22: LED, LED_SMD:LED_0603_1608Metric, F.Cu at (145.5, 160.9)
- added D23: LED, LED_SMD:LED_0603_1608Metric, F.Cu at (161.0, 150.4)
- added D24: LED, LED_SMD:LED_0603_1608Metric, F.Cu at (158.6, 166.8)
- added D25: LTST-C193KFKT-5A, LED_SMD:LED_0603_1608Metric, F.Cu at (145.3, 172.3)
- added D27: D_Schottky, Diode_SMD:D_SOD-123, B.Cu at (181.3, 115.6)
- added D28: TPD2EUSB30DRTR, LHRS_ICs:TPD2EUSB30DRTR, B.Cu at (184.9, 116.0)
- added F2: Fuse, FuseHolder:FUSE_3568, F.Cu at (130.8, 67.3)
- added IC7: ISO1042QDWRQ1, ISO1042QDWRQ1:ISO1042QDWRQ1, F.Cu at (248.9, 91.7)
- added J13: USB_C_Receptacle_USB2.0_16P, LHRS_Connectors:USB_C_Receptacle_GCT_USB4105-xx-A_16P_TopMnt_Horizontal, F.Cu at (186.7, 116.0)
- added J4: Thermistor, Connector_Molex:Molex_Nano-Fit_105313-xx02_1x02_P2.50mm_Horizontal, F.Cu at (170.1, 60.9)
- added J7: MotorConn_1, Connector_Molex:Molex_Nano-Fit_105314-xx10_2x05_P2.50mm_Horizontal, F.Cu at (176.3, 86.0)
- added J8: Motor_Conn2, Connector_Molex:Molex_Nano-Fit_105314-xx14_2x07_P2.50mm_Horizontal, F.Cu at (176.3, 65.0)
- added Q5: IRLML2030TRPBF, IRLML2030TRPBF:IRLML2030TRPBF, F.Cu at (126.3, 175.2)
- added Q6: IRLML2030TRPBF, IRLML2030TRPBF:IRLML2030TRPBF, F.Cu at (142.2, 161.3)
- added Q7: IRLML2030TRPBF, IRLML2030TRPBF:IRLML2030TRPBF, F.Cu at (157.1, 150.3)
- added Q8: IRLML2030TRPBF, IRLML2030TRPBF:IRLML2030TRPBF, F.Cu at (158.8, 163.2)
- added R13: 60, Resistor_SMD:R_0603_1608Metric_Pad0.98x0.95mm_HandSolder, B.Cu at (225.7, 86.4)
- added R23: 100k, Resistor_SMD:R_0603_1608Metric_Pad0.98x0.95mm_HandSolder, F.Cu at (85.3, 175.5)
- added R32: 120, Resistor_SMD:R_0603_1608Metric_Pad0.98x0.95mm_HandSolder, F.Cu at (45.0, 117.4)
- added R51: 10k, Resistor_SMD:R_0603_1608Metric_Pad0.98x0.95mm_HandSolder, B.Cu at (236.9, 127.0)
- added R52: 60, Resistor_SMD:R_0603_1608Metric_Pad0.98x0.95mm_HandSolder, B.Cu at (247.7, 98.7)
- added R53: 1k, Resistor_SMD:R_0603_1608Metric_Pad0.98x0.95mm_HandSolder, F.Cu at (127.7, 172.1)
- added R56: 1k, Resistor_SMD:R_0603_1608Metric_Pad0.98x0.95mm_HandSolder, F.Cu at (159.1, 160.2)
- added R57: 60, Resistor_SMD:R_0603_1608Metric_Pad0.98x0.95mm_HandSolder, B.Cu at (251.1, 98.7)
- added R58: 10k, Resistor_SMD:R_0603_1608Metric_Pad0.98x0.95mm_HandSolder, B.Cu at (239.5, 123.6)
- added R59: 10k, Resistor_SMD:R_0603_1608Metric_Pad0.98x0.95mm_HandSolder, B.Cu at (239.5, 126.9)
- added R60: 5k, Resistor_SMD:R_0603_1608Metric_Pad0.98x0.95mm_HandSolder, F.Cu at (145.2, 170.8)
- added R61: 5.1k, Resistor_SMD:R_0603_1608Metric_Pad0.98x0.95mm_HandSolder, F.Cu at (240.5, 103.9)
- added R62: 9.1k, Resistor_SMD:R_0603_1608Metric_Pad0.98x0.95mm_HandSolder, F.Cu at (240.5, 106.4)
- added R66: 5.1k, Resistor_SMD:R_0603_1608Metric_Pad0.98x0.95mm_HandSolder, B.Cu at (185.6, 117.5)
- added R67: 5.1k, Resistor_SMD:R_0603_1608Metric_Pad0.98x0.95mm_HandSolder, B.Cu at (185.6, 114.5)
- added TP10: TestPoint, TestPoint:TestPoint_Loop_D2.50mm_Drill1.0mm_LowProfile, F.Cu at (37.8, 65.9)
- added TP11: TestPoint, TestPoint:TestPoint_Loop_D2.50mm_Drill1.0mm_LowProfile, F.Cu at (37.8, 70.5)
- added TP12: TestPoint, TestPoint:TestPoint_Loop_D2.50mm_Drill1.0mm_LowProfile, F.Cu at (37.8, 75.2)
- added TP13: TestPoint, TestPoint:TestPoint_Loop_D2.50mm_Drill1.0mm_LowProfile, F.Cu at (37.8, 79.8)
- added TP14: TestPoint, TestPoint:TestPoint_Loop_D2.50mm_Drill1.0mm_LowProfile, F.Cu at (37.8, 84.5)
- added TP15: TestPoint, TestPoint:TestPoint_Loop_D2.50mm_Drill1.0mm_LowProfile, F.Cu at (37.8, 89.2)
- added TP16: TestPoint, TestPoint:TestPoint_Loop_D2.50mm_Drill1.0mm_LowProfile, F.Cu at (42.5, 65.9)
- added TP17: TestPoint, TestPoint:TestPoint_Loop_D2.50mm_Drill1.0mm_LowProfile, F.Cu at (42.5, 70.5)
- added TP18: TestPoint, TestPoint:TestPoint_Loop_D2.50mm_Drill1.0mm_LowProfile, F.Cu at (42.5, 75.2)
- added TP19: TestPoint, TestPoint:TestPoint_Loop_D2.50mm_Drill1.0mm_LowProfile, F.Cu at (42.5, 79.8)
- added TP20: TestPoint, TestPoint:TestPoint_Loop_D2.50mm_Drill1.0mm_LowProfile, F.Cu at (42.5, 84.5)
- added TP21: TestPoint, TestPoint:TestPoint_Loop_D2.50mm_Drill1.0mm_LowProfile, F.Cu at (42.5, 89.2)
- added TP22: TestPoint, TestPoint:TestPoint_Loop_D2.50mm_Drill1.0mm_LowProfile, F.Cu at (47.1, 65.9)
- added TP23: TestPoint, TestPoint:TestPoint_Loop_D2.50mm_Drill1.0mm_LowProfile, F.Cu at (47.1, 70.5)
- added TP24: TestPoint, TestPoint:TestPoint_Loop_D2.50mm_Drill1.0mm_LowProfile, F.Cu at (47.1, 75.2)
- added TP25: TestPoint, TestPoint:TestPoint_Loop_D2.50mm_Drill1.0mm_LowProfile, F.Cu at (47.1, 79.8)
- added TP26: TestPoint, TestPoint:TestPoint_Loop_D2.50mm_Drill1.0mm_LowProfile, F.Cu at (47.1, 84.5)
- added TP27: TestPoint, TestPoint:TestPoint_Loop_D2.50mm_Drill1.0mm_LowProfile, F.Cu at (47.1, 89.2)
- added TP28: TestPoint, TestPoint:TestPoint_Loop_D2.50mm_Drill1.0mm_LowProfile, F.Cu at (51.8, 65.9)
- added TP29: TestPoint, TestPoint:TestPoint_Loop_D2.50mm_Drill1.0mm_LowProfile, F.Cu at (51.8, 70.5)
- added TP30: TestPoint, TestPoint:TestPoint_Loop_D2.50mm_Drill1.0mm_LowProfile, F.Cu at (51.8, 75.2)
- added TP31: TestPoint, TestPoint:TestPoint_Loop_D2.50mm_Drill1.0mm_LowProfile, F.Cu at (51.8, 79.8)
- added TP32: TestPoint, TestPoint:TestPoint_Loop_D2.50mm_Drill1.0mm_LowProfile, F.Cu at (51.8, 84.5)
- added TP33: TestPoint, TestPoint:TestPoint_Loop_D2.50mm_Drill1.0mm_LowProfile, F.Cu at (51.8, 89.2)
- added TP34: TestPoint, TestPoint:TestPoint_Loop_D2.50mm_Drill1.0mm_LowProfile, F.Cu at (56.4, 65.9)
- added TP35: TestPoint, TestPoint:TestPoint_Loop_D2.50mm_Drill1.0mm_LowProfile, F.Cu at (56.4, 70.5)
- added TP36: TestPoint, TestPoint:TestPoint_Loop_D2.50mm_Drill1.0mm_LowProfile, F.Cu at (56.4, 75.2)
- added TP37: TestPoint, TestPoint:TestPoint_Loop_D2.50mm_Drill1.0mm_LowProfile, F.Cu at (56.4, 79.8)
- added TP38: TestPoint, TestPoint:TestPoint_Loop_D2.50mm_Drill1.0mm_LowProfile, F.Cu at (56.4, 84.5)
- C20, C21, C22, C23, C37, C39, D4, IC3, JP5, R14, R35, R38, R42, TP5, TP6, TP7, TP8, TP9: moved to B.Cu
- C40: value 0.1u -> 1uF; moved to B.Cu
- C41: value 10uF -> 0.1u; moved to B.Cu
- C42: value 2.2uF -> 10u; moved to B.Cu
- C43: value 2.2uF -> .1u; moved to B.Cu
- C44: value 10u -> 4.7uF
- C45: value .1u -> 330pF; moved to B.Cu
- C46: value 10uF -> 330pF; footprint Capacitor_SMD:C_0805_2012Metric -> Capacitor_SMD:C_0603_1608Metric_Pad1.08x0.95mm_HandSolder; moved to B.Cu
- D15, D16: value D_Schottky -> LED; footprint VSSAF522-M3_H:SODFL5226X100N -> LED_SMD:LED_0603_1608Metric
- D17, D18: value LED -> D_Schottky; footprint LED_SMD:LED_0603_1608Metric -> VSSAF522-M3_H:SODFL5226X100N; moved to B.Cu
- D20: value D_Schottky -> LED; footprint Diode_SMD:D_SOD-123 -> LED_SMD:LED_0603_1608Metric
- D21: value TPD2EUSB30DRTR -> LED; footprint LHRS_ICs:TPD2EUSB30DRTR -> LED_SMD:LED_0603_1608Metric
- IC4: value ISO1042QDWRQ1 -> ISO7741DWR; footprint ISO1042QDWRQ1:ISO1042QDWRQ1 -> ISO7741DWR:ISO7741DWR
- J11: renamed from J9; moved to F.Cu
- J2: value CAN_NANO_01x03 -> WaveSculptor Debug; footprint LHRS_Connectors:Molex_Nano-Fit_105309-xx03_1x03_P2.50mm_Vertical -> LHRS_Connectors:Molex_Nano-Fit_105309-xx04_1x04_P2.50mm_Vertical
- J5: value Motor_Conn1 -> CAN_NANO_01x03; footprint Connector_Molex:Molex_Nano-Fit_105314-xx12_2x06_P2.50mm_Horizontal -> LHRS_Connectors:Molex_Nano-Fit_105309-xx03_1x03_P2.50mm_Vertical
- JP2: value SolderJumper_2_Bridged -> SolderJumper_2_Open; footprint Jumper:SolderJumper-2_P1.3mm_Bridged2Bar_RoundedPad1.0x1.5mm -> Jumper:SolderJumper-2_P1.3mm_Open_RoundedPad1.0x1.5mm; moved to B.Cu
- JP3: value SolderJumper_2_Open -> SolderJumper_2_Bridged; footprint Jumper:SolderJumper-2_P1.3mm_Open_RoundedPad1.0x1.5mm -> Jumper:SolderJumper-2_P1.3mm_Bridged2Bar_RoundedPad1.0x1.5mm; moved to B.Cu
- L2: value 10u -> 10uH
- Q3: value IRLML2030TRPBF -> DMP3099L-7; footprint IRLML2030TRPBF:IRLML2030TRPBF -> DMP3099L-7:DMP3099L-7
- R24: value 100k -> 120
- R25: value 120 -> 2k
- R26: value 2k -> 120
- R36, R40: value 33k -> 10k; moved to B.Cu
- R37: value 5k -> 33k; moved to B.Cu
- R39: value 10k -> 5k; moved to B.Cu
- R41: value 10k -> 33k; moved to B.Cu
- R43, R44: value 60 -> 10k; moved to B.Cu
- R45, R46: value 10k -> 1k
- R47: value R -> 10k; moved to B.Cu
- R48: value 1k -> 10k; moved to B.Cu
- R49: value 5.1k -> 10k; moved to B.Cu
- R50: value 9.1k -> 10k; moved to B.Cu
- R54, R55: value 5.1k -> 1k
- U5: value MCP4822 -> MCP4922T-E/ST; footprint MCP4822T-E_SN:MCP4822T-E_SN -> MCP4922T-EST:MCP4922T-EST
- moved C23 318.2 mm to (229.8, 87.4), turned to -90 degrees
- moved C21 316.6 mm to (228.2, 83.8), turned to 90 degrees
- moved R14 316.5 mm to (228.2, 87.3), turned to 90 degrees
- moved C41 313.8 mm to (251.1, 100.3)
- moved C22 310.8 mm to (222.4, 83.8), turned to 90 degrees
- moved JP1 310.5 mm to (226.6, 88.4), turned to -90 degrees
- moved C20 309.4 mm to (230.2, 83.8), turned to 90 degrees
- moved IC2 307.3 mm to (225.4, 83.8)
- moved C42 305.4 mm to (234.5, 122.8), turned to 180 degrees
- moved D4 304.6 mm to (225.4, 83.8), turned to 180 degrees
- moved C43 304.5 mm to (233.6, 125.2), turned to 90 degrees
- moved IC4 304.5 mm to (232.0, 104.5)
- moved IC5 304.2 mm to (232.0, 115.6)
- moved JP2 303.3 mm to (242.1, 125.4), turned to 180 degrees
- moved JP3 302.8 mm to (242.0, 127.9), turned to 180 degrees
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- renumbered D19 to D26, J8 to J10, J10 to J12, J4 to J6, J7 to J9, R11 to R10, R12 to R11, R13 to R12, R16 to R15, R17 to R16, R18 to R17, R19 to R18, R20 to R19, R4 to R2, R21 to R20, R22 to R21, R23 to R22, R32 to R33, R33 to R34, R5 to R4, R6 to R5, R7 to R6, R51 to R63, R52 to R64, R53 to R65, R8 to R7, R9 to R8, R10 to R9
Connections:
- C38 pad 1: +3.3V -> GND
- C38 pad 2: GND -> /+TH
- C40 pad 1: Net-(JP2-B) -> +3.3V
- C40 pad 2: GND_ISO -> GND
- C41 pad 1: +3.3V -> Net-(JP4-B)
- C41 pad 2: GND -> GND_ISO
- C42 pad 1: /Motor Comms/+3.3V_ISO -> GND_ISO
- C42 pad 2: Net-(JP5-B) -> /Motor Comms/+5V_ISO
- C43 pad 2: GND -> /Motor Comms/+5V_ISO
- C44 pad 1: GND_ISO -> /Motor Comms/+3.3V_in
- C44 pad 2: /Motor Comms/+3.3V_ISO -> GND
- C45 pad 1: GND_ISO -> /Motor Comms/+5V_ISO
- C45 pad 2: /Motor Comms/+3.3V_ISO -> /Motor Comms/+3.3V_in
- C46 pad 1: GND -> GND_ISO
- C46 pad 2: /MCU + Peripherals/+5V_USB -> GND
- C5 pad 1: /+12V_Fan -> /Power Regulation/12VBuck/V_in
- C8 pad 1: /+12V_Fan -> /Power Regulation/12VBuck/V_in
- C9 pad 1: /+12V_Fan -> /Power Regulation/12VBuck/V_in
- D15 pad 1: /+12V_Fan -> Net-(D15-K)
- D15 pad 2: GND -> /MCU + Peripherals/SW_LED3
- D16 pad 1: /+12V_Fan -> Net-(D16-K)
- D16 pad 2: GND -> /MCU + Peripherals/SW_LED4
- D17 pad 1: GND -> /+12V_PP
- D17 pad 2: Net-(D17-A) -> GND
- D18 pad 1: GND -> /+12V_PP
- D18 pad 2: Net-(D18-A) -> GND
- D20 pad 1: /MCU + Peripherals/+5V_USB -> GND_ISO
- D20 pad 2: /MCU + Peripherals/USB-C Connector/VBUS_IN -> Net-(D20-A)
- D21 pad 1: /MCU + Peripherals/100PinMCU/USB_DP -> GND_ISO
- D21 pad 2: /MCU + Peripherals/100PinMCU/USB_DM -> Net-(D21-A)
- IC4 pad 10: GND_ISO -> Net-(IC4-EN2)
- IC4 pad 11: /Motor Comms/+3.3V_ISO -> /Motor Comms/Pulse_ADC_DIV
- IC4 pad 12: /MTR_CANL -> /Motor Comms/Map_Bit0_Gate
- IC4 pad 13: /MTR_CANH -> /Motor Comms/F/R_Mode_Gate
- IC4 pad 14: unconnected-(IC4-NC_4-Pad14) -> /Motor Comms/PwrMode_Gate
- IC4 pad 16: /Motor Comms/+3.3V_ISO -> /Motor Comms/+5V_ISO
- IC4 pad 3: /MCU + Peripherals/MtrCAN_TX -> /MCU + Peripherals/PWR_EN
- IC4 pad 4: unconnected-(IC4-NC_1-Pad4) -> /MCU + Peripherals/FWD_EN
- IC4 pad 5: /MCU + Peripherals/MtrCAN_RX -> /map_bit0
- IC4 pad 6: unconnected-(IC4-NC_2-Pad6) -> /MCU + Peripherals/Pulse_ADC4
- IC4 pad 7: unconnected-(IC4-NC_3-Pad7) -> Net-(IC4-EN1)
- IC5 pad 12: unconnected-(IC5-OUTC-Pad12) -> /Motor Comms/Map_Bit3_Gate
- IC5 pad 13: /Motor Comms/F/R_Mode_Gate -> /Motor Comms/Map_Bit2_Gate
- IC5 pad 14: /Motor Comms/PwrMode_Gate -> /Motor Comms/Map_Bit1_Gate
- IC5 pad 16: /Motor Comms/+3.3V_ISO -> /Motor Comms/+5V_ISO
- IC5 pad 3: /MCU + Peripherals/PWR_EN -> /map_bit1
- IC5 pad 4: /MCU + Peripherals/FWD_EN -> /map_bit2
- IC5 pad 5: unconnected-(IC5-INC-Pad5) -> /map_bit3
- IC6 pad 12: /Motor Comms/SPI_CS_ISO -> /Motor Comms/SPI_MOSI_ISO
- IC6 pad 13: /Motor Comms/SPI_MOSI_ISO -> /Motor Comms/SPI_CLK_ISO
- IC6 pad 14: /Motor Comms/SPI_CLK_ISO -> /Motor Comms/SPI_CS_ISO
- IC6 pad 16: /Motor Comms/+3.3V_ISO -> /Motor Comms/+5V_ISO
- IC6 pad 3: /MCU + Peripherals/DAC_CLK -> /MCU + Peripherals/DAC_CS
- IC6 pad 4: /MCU + Peripherals/DAC_MOSI -> /MCU + Peripherals/DAC_CLK
- IC6 pad 5: /MCU + Peripherals/DAC_CS -> /MCU + Peripherals/DAC_MOSI
- J2 pad 1: /CarCAN_H -> /+12V_PP
- J2 pad 2: /CarCAN_L -> /MTR_CANH
- J2 pad 3: Net-(J2-SHIELD) -> /MTR_CANL
- J5 pad 1: /Accel_ADC -> /CarCAN_H
- J5 pad 2: /BrakeADC -> /CarCAN_L
- J5 pad 3: /MTR_CANH -> Net-(J3-SHIELD)
- J6 pad 1: +12V -> /+12V_PP
- J9 pad 1: GND -> /+12V_PP
- J9 pad 2: /FAN2_PWM -> /FAN2_TACH
- J9 pad 3: /FAN2_TACH -> /FAN2_PWM
- J9 pad 4: +12V -> GND
- JP2 pad 1: Net-(JP2-A) -> /MCU + Peripherals/LDAC
- JP3 pad 1: /MCU + Peripherals/LDAC -> GND
- JP3 pad 2: Net-(JP3-B) -> Net-(JP2-B)
- JP4 pad 1: GND -> Net-(JP4-A)
- JP4 pad 2: Net-(JP3-B) -> Net-(JP4-B)
- JP5 pad 2: Net-(JP5-B) -> /Motor Comms/+3.3V_in
- L2 pad 1: Net-(JP5-B) -> +3.3V
- L2 pad 2: +3.3V -> /Motor Comms/+3.3V_in
- PS1 pad 2: Net-(JP5-B) -> /Motor Comms/+3.3V_in
- PS1 pad 4: /Motor Comms/+3.3V_ISO -> /Motor Comms/+5V_ISO
- Q2 pad 5: /+12V_Fan -> /Power Regulation/12VBuck/V_in
- Q3 pad 1: /PWR_MODE_IN -> /PWR_MODE_OUT
- Q3 pad 3: /PWR_MODE_OUT -> /PWR_MODE_IN
- R1 pad 1: Net-(J2-SHIELD) -> Net-(J3-SHIELD)
- R14 pad 1: /CarCAN_H -> Net-(C23-Pad2)
- R14 pad 2: Net-(C23-Pad2) -> Net-(JP1-A)
- R24 pad 1: /+TH -> Net-(D8-K)
- R24 pad 2: +3.3V -> GND
- R25 pad 1: Net-(D8-K) -> Net-(D9-K)
- R26 pad 1: Net-(D9-K) -> Net-(D10-K)
- R27 pad 1: Net-(D10-K) -> Net-(D11-K)
- R28 pad 1: Net-(D11-K) -> Net-(D12-K)
- R29 pad 1: Net-(D12-K) -> Net-(D13-K)
- R3 pad 1: Net-(J5-Pin_6) -> Net-(J8-Pin_7)
- R30 pad 1: Net-(D13-K) -> Net-(D14-K)
- R31 pad 1: Net-(D14-K) -> Net-(D15-K)
- R35 pad 2: /MCU + Peripherals/SCL -> /MCU + Peripherals/SDA
- R36 pad 2: Net-(IC3-ADDR_SEL) -> /MCU + Peripherals/SCL
- R37 pad 1: /FAN1_TACH -> +3.3V
- R37 pad 2: +3.3V -> Net-(IC3-ADDR_SEL)
- R38 pad 1: /FAN2_TACH -> /FAN1_TACH
- R39 pad 1: +3.3V -> /FAN2_TACH
- R39 pad 2: /MCU + Peripherals/ALERT -> +3.3V
- R40 pad 2: Net-(IC3-CLK) -> /MCU + Peripherals/ALERT
- R41 pad 2: Net-(IC5-EN1) -> Net-(IC3-CLK)
- R42 pad 2: Net-(IC6-EN1) -> Net-(IC4-EN1)
- R43 pad 1: /MTR_CANH -> +3.3V
- R43 pad 2: Net-(JP2-A) -> Net-(IC5-EN1)
- R44 pad 1: Net-(JP2-B) -> +3.3V
- R44 pad 2: /MTR_CANL -> Net-(IC6-EN1)
- R45 pad 1: /Motor Comms/+3.3V_ISO -> Net-(D19-A)
- R45 pad 2: Net-(IC5-EN2) -> /Motor Comms/PwrMode_Gate
- R46 pad 1: /Motor Comms/+3.3V_ISO -> Net-(D20-A)
- R46 pad 2: Net-(IC6-EN2) -> /Motor Comms/F/R_Mode_Gate
- R47 pad 1: Net-(D17-A) -> /Motor Comms/+5V_ISO
- R47 pad 2: /Motor Comms/PwrMode_Gate -> Net-(IC4-EN2)
- R48 pad 1: Net-(D18-A) -> /Motor Comms/+5V_ISO
- R48 pad 2: /Motor Comms/F/R_Mode_Gate -> Net-(IC5-EN2)
- R49 pad 1: /MCU + Peripherals/Pulse_ADC4 -> /Motor Comms/+5V_ISO
- R49 pad 2: /Mtr_Pulse -> Net-(IC6-EN2)
- R50 pad 1: /MCU + Peripherals/Pulse_ADC4 -> Net-(U5-~{SHDN})
- R50 pad 2: GND -> /Motor Comms/+5V_ISO
- R54 pad 1: GND -> Net-(D22-A)
- R54 pad 2: /MCU + Peripherals/USB-C Connector/CC1 -> /Motor Comms/Map_Bit1_Gate
- R55 pad 1: GND -> Net-(D23-A)
- R55 pad 2: /MCU + Peripherals/USB-C Connector/CC2 -> /Motor Comms/Map_Bit2_Gate
- TP1 pad 1: /+12V_Fan -> /Power Regulation/12VBuck/V_in
- U1 pad 2: /+12V_Fan -> /Power Regulation/12VBuck/V_in
- U1 pad 3: /+12V_Fan -> /Power Regulation/12VBuck/V_in
- U4 pad 16: GND -> /MCU + Peripherals/100PinMCU/PC1
- U4 pad 84: /MCU + Peripherals/100PinMCU/PD2 -> /MCU + Peripherals/SW_LED4
- U4 pad 85: /MCU + Peripherals/100PinMCU/PD3 -> /MCU + Peripherals/SW_LED3
- U5 pad 1: /Motor Comms/+3.3V_ISO -> /Motor Comms/+5V_ISO
- U5 pad 2: /Motor Comms/SPI_CS_ISO -> unconnected-(U5-NC-Pad2)
- U5 pad 3: /Motor Comms/SPI_CLK_ISO -> /Motor Comms/SPI_CS_ISO
- U5 pad 4: /Motor Comms/SPI_MOSI_ISO -> /Motor Comms/SPI_CLK_ISO
- U5 pad 5: Net-(JP3-B) -> /Motor Comms/SPI_MOSI_ISO
- U5 pad 6: /BrakeADC -> unconnected-(U5-NC-Pad6)
- U5 pad 7: GND_ISO -> unconnected-(U5-NC-Pad7)
- U5 pad 8: /Accel_ADC -> Net-(JP2-B)
Routing:
- net /Motor Comms/SPI_CS_ISO: track 0.00 -> 2.93 mm
- net /Motor Comms/SPI_MOSI_ISO: track 0.00 -> 2.71 mm
- net /Motor Comms/SPI_CLK_ISO: track 0.00 -> 2.67 mm
Other:
- board size 90 x 60 mm -> 100 x 80 mm

Commit message: final layout
Parts:
- C38, R22, R23, R24, R25, R26, R27, R28, R29, R30, R31, R32, R45, R46, R53, R54, R55, R56, R60, R61, R62: moved to B.Cu
- J7: footprint Connector_Molex:Molex_Nano-Fit_105314-xx10_2x05_P2.50mm_Horizontal -> LHRS_Connectors:Molex_Nano-Fit_105314-xx10_2x05_P2.50mm_Horizontal
- J8: footprint Connector_Molex:Molex_Nano-Fit_105314-xx14_2x07_P2.50mm_Horizontal -> cutom_2x7_nanofit:nanofit_2x7_diff_pinouts
- moved R23 141.5 mm to (171.3, 63.1), turned to 180 degrees
- moved C23 133.3 mm to (100.2, 118.5), turned to 180 degrees
- moved R14 131.3 mm to (100.2, 116.9), turned to 0 degrees
- moved C20 131.2 mm to (103.8, 118.9), turned to 0 degrees
- moved TP9 131.2 mm to (159.8, 73.2), turned to 90 degrees
- moved C21 128.8 mm to (103.8, 116.9), turned to 0 degrees
- moved R13 127.7 mm to (101.2, 114.4), turned to -90 degrees
- moved TP8 126.8 mm to (159.8, 69.8), turned to -90 degrees
- moved TP7 126.0 mm to (162.8, 71.5), turned to -90 degrees
- moved D4 125.4 mm to (103.8, 114.1), turned to 90 degrees
- moved IC2 125.4 mm to (103.8, 114.1), turned to -90 degrees
- moved TP37 125.2 mm to (175.5, 118.5)
- moved TP38 125.2 mm to (175.5, 123.2)
- moved TP13 124.4 mm to (156.8, 116.0)
- moved TP19 124.4 mm to (161.5, 116.0)
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Connections:
- J7 pad 4: /BrakeADC -> /Mtr_Pulse
- J7 pad 8: /Mtr_Pulse -> /BrakeADC
- J8 pad 10: /MTR_CANL -> /map_bit1_sig
- J8 pad 13: /FR_MODE_OUT -> /PWR_MODE_OUT
- J8 pad 2: /map_bit0_sig -> /PWR_MODE_IN
- J8 pad 3: /map_bit1_sig -> /FR_MODE_OUT
- J8 pad 4: /map_bit2_sig -> /MTR_CANL
- J8 pad 5: /map_bit3_sig -> /map_bit0_sig
- J8 pad 6: /PWR_MODE_IN -> /map_bit2_sig
- J8 pad 9: /PWR_MODE_OUT -> /map_bit3_sig

Commit message: layoutttttttttttttttttttttttttttttttttttt
Parts:
- removed TP10, TP11, TP12, TP13, TP14, TP15, TP16, TP17, TP18, TP19, TP20, TP21, TP22, TP23, TP24, TP25, TP26, TP27, TP28, TP29, TP30, TP31, TP32, TP33, TP34, TP35, TP36, TP37, TP38: TestPoint, TestPoint:TestPoint_Loop_D2.50mm_Drill1.0mm_LowProfile
- added C49: 4.7nF, Capacitor_SMD:C_0603_1608Metric_Pad1.08x0.95mm_HandSolder, B.Cu at (94.8, 95.8)
- added D17: LED, LED_SMD:LED_0603_1608Metric, F.Cu at (129.9, 77.4)
- added D18: LED, LED_SMD:LED_0603_1608Metric, F.Cu at (133.3, 92.9)
- added D19: LED, LED_SMD:LED_0603_1608Metric, F.Cu at (133.3, 96.0)
- added D20: LED, LED_SMD:LED_0603_1608Metric, F.Cu at (133.2, 99.0)
- added D21: LED, LED_SMD:LED_0603_1608Metric, F.Cu at (133.2, 101.9)
- added J13: Debug_Conn, Connector_PinHeader_2.54mm:PinHeader_2x15_P2.54mm_Vertical, F.Cu at (101.3, 127.3)
- added R33: 250, Resistor_SMD:R_0603_1608Metric_Pad0.98x0.95mm_HandSolder, B.Cu at (129.7, 77.5)
- added R34: 250, Resistor_SMD:R_0603_1608Metric_Pad0.98x0.95mm_HandSolder, B.Cu at (133.3, 93.0)
- added R35: 250, Resistor_SMD:R_0603_1608Metric_Pad0.98x0.95mm_HandSolder, B.Cu at (133.3, 96.1)
- added R36: 250, Resistor_SMD:R_0603_1608Metric_Pad0.98x0.95mm_HandSolder, B.Cu at (133.3, 99.2)
- added R37: 250, Resistor_SMD:R_0603_1608Metric_Pad0.98x0.95mm_HandSolder, B.Cu at (133.3, 102.2)
- added R71: 1M, Resistor_SMD:R_0603_1608Metric_Pad0.98x0.95mm_HandSolder, F.Cu at (94.8, 95.8)
- C44, JP4: moved to B.Cu
- CR1, J12: moved to F.Cu
- D31: renamed from D26; moved to F.Cu
- D33: renamed from D28; moved to F.Cu
- R24, R26, R27, R28, R29, R30, R31, R32: value 120 -> 250
- R39: renamed from R34; moved to F.Cu
- R68: renamed from R63; moved to B.Cu
- moved J14 94.2 mm to (93.6, 101.8), turned to -90 degrees
- moved R72 92.5 mm to (94.7, 100.3), turned to 0 degrees
- moved R73 91.6 mm to (94.7, 103.3), turned to 0 degrees
- moved SW1 89.8 mm to (95.5, 112.8), turned to 90 degrees
- moved D5 89.8 mm to (95.4, 112.8), turned to 180 degrees
- moved D33 86.8 mm to (99.2, 101.8)
- moved D32 82.8 mm to (99.5, 103.0), turned to -90 degrees
- moved C50 82.2 mm to (99.5, 104.2), turned to 90 degrees
- moved J2 79.8 mm to (186.2, 110.1), turned to 0 degrees
- moved C30 78.2 mm to (102.0, 117.2), turned to 0 degrees
- moved R15 77.6 mm to (102.0, 115.6), turned to 0 degrees
- moved D7 75.6 mm to (102.3, 109.5), turned to 180 degrees
- moved R22 75.5 mm to (102.4, 109.4), turned to 180 degrees
- moved Reset1 74.5 mm to (103.3, 114.2), turned to -90 degrees
- moved J3 67.5 mm to (161.6, 126.8), turned to -90 degrees
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- renumbered C49 to C50, D17 to D22, D18 to D23, D20 to D24, D19 to D25, D21 to D26, D22 to D27, D23 to D28, D24 to D29, D25 to D30, D27 to D32, J13 to J14, Q4 to Q3, Q3 to Q4, R33 to R38, R35 to R40, R36 to R41, R37 to R42, R38 to R43, R39 to R44, R40 to R45, R41 to R46, R42 to R47, R43 to R48, R44 to R49, R46 to R50, R45 to R51, R47 to R52, R48 to R53, R49 to R54, R50 to R55, R51 to R56, R52 to R57, R53 to R58, R54 to R59, R55 to R60, R56 to R61, R57 to R62, R58 to R63, R59 to R64, R60 to R65, R61 to R66, R62 to R67, R64 to R69, R65 to R70, R66 to R72, R67 to R73
Connections:
- D13 pad 2: /MCU + Peripherals/SW_LED1 -> /MCU + Peripherals/HB_LED
- D14 pad 2: /MCU + Peripherals/SW_LED2 -> /MCU + Peripherals/Mtr_Fault
- D15 pad 2: /MCU + Peripherals/SW_LED3 -> /MCU + Peripherals/BPS_Fault
- D16 pad 2: /MCU + Peripherals/SW_LED4 -> /MCU + Peripherals/ESTOP_Fault
- J14 pad S1: GND -> Net-(J14-SHIELD)
- J14 pad S2: GND -> Net-(J14-SHIELD)
- J14 pad S3: GND -> Net-(J14-SHIELD)
- J14 pad S4: GND -> Net-(J14-SHIELD)
Routing:
- net Net-(JP1-A): track 0.00 -> 14.8 mm
- net /CarCAN_L: track 0.00 -> 10.1 mm, vias 0 -> 2
- net Net-(J10-Pin_3): track 0.00 -> 8.21 mm
- net /CarCAN_H: track 0.00 -> 6.22 mm, vias 0 -> 1
- net Net-(J10-Pin_4): track 0.00 -> 5.77 mm
- net Net-(C23-Pad2): track 0.00 -> 4.04 mm
- net /Power Regulation/12VBuck/V_in: vias 0 -> 8
Other:
- board text added: "Galvanic Isolation"
- board text added: "MoCo Conn 1"
- board text added: "MoCo Conn 2"

Commit message: migtve finally lcokeefd in = ggs
Parts:
- removed TP5, TP6, TP7, TP8, TP9: TestPoint, diddle_shah:TestPoint_HEX_3mmID
- added J14: Debug_Conn1, Connector_PinHeader_2.54mm:PinHeader_2x08_P2.54mm_Vertical, F.Cu at (131.9, 127.2)
- added J15: Debug_Conn2, Connector_PinHeader_2.54mm:PinHeader_2x06_P2.54mm_Vertical, F.Cu at (165.9, 127.3)
- added JP6: SolderJumper_2_Open, Jumper:SolderJumper-2_P1.3mm_Open_RoundedPad1.0x1.5mm, F.Cu at (116.7, 61.6)
- C1, C11, C12, C13, C5, C50, C7: moved to B.Cu
- C2, C27, C28, C31, C32, C33, C35, C36, C39, C40, C8, C9, D4, IC3, R10, R11, R16, R17, R4, R40, R41, R45, R46, R5, R6, R69, R7, R72, R73, R8, R9: moved to F.Cu
- F1, F2: footprint FuseHolder:FUSE_3568 -> LHRS_Power:Fuse-3557-2
- J13: value Debug_Conn -> Fan_Debug_Conn; footprint Connector_PinHeader_2.54mm:PinHeader_2x15_P2.54mm_Vertical -> Connector_PinHeader_2.54mm:PinHeader_1x05_P2.54mm_Vertical
- J4: footprint Connector_Molex:Molex_Nano-Fit_105313-xx02_1x02_P2.50mm_Horizontal -> LHRS_Connectors:Molex_Nano-Fit_105309-xx02_1x02_P2.50mm_Vertical
- J6, J9: footprint LHRS_Connectors:Molex_Nano-Fit_105313-xx04_1x04_P2.50mm_Horizontal -> LHRS_Connectors:Molex_Nano-Fit_105309-xx04_1x04_P2.50mm_Vertical
- J7: footprint LHRS_Connectors:Molex_Nano-Fit_105314-xx10_2x05_P2.50mm_Horizontal -> LHRS_Connectors:Molex_Nano-Fit_105310-xx10_2x05_P2.50mm_Vertical
- J8: footprint cutom_2x7_nanofit:nanofit_2x7_diff_pinouts -> cutom_2x7_nanofit:custom_2x07_vertical_nanofit
- PS1: value ROE-3.305S -> ROE-3.505S
- moved J3 93.5 mm to (103.0, 54.0), turned to 90 degrees
- moved J1 83.3 mm to (132.7, 54.2), turned to 90 degrees
- moved R1 82.5 mm to (112.0, 52.1), turned to 90 degrees
- moved J5 79.8 mm to (116.0, 54.0), turned to 90 degrees
- moved D23 67.2 mm to (98.0, 82.2), turned to -90 degrees
- moved J4 66.8 mm to (158.9, 126.7), turned to -90 degrees
- moved J9 66.4 mm to (93.9, 83.1), turned to 180 degrees
- moved R23 62.7 mm to (159.4, 124.7), turned to 0 degrees
- moved C40 57.4 mm to (98.1, 71.0), turned to 180 degrees
- moved R42 56.1 mm to (96.4, 74.0), turned to 0 degrees
- moved C39 56.0 mm to (98.1, 72.5), turned to 180 degrees
- moved R43 54.7 mm to (96.4, 75.5), turned to 180 degrees
- moved R41 54.3 mm to (101.5, 71.0), turned to 0 degrees
- moved R44 53.3 mm to (96.4, 77.0), turned to 180 degrees
- moved R40 53.0 mm to (101.5, 72.5), turned to 0 degrees
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- renumbered J14 to J16
Connections:
- net /Motor Comms/+3.3V_in renamed /Motor Comms/+5V_in
- net /Power Regulation/12VBuck/V_in renamed /Power Regulation/Vout_pp
- C17 pad 1: /Power Regulation/LDO/Vin -> +5V
- D3 pad 2: /Power Regulation/LDO/Vin -> +5V
- J13 pad 1: +3.3V -> /MCU + Peripherals/ALERT
- J13 pad 2: GND -> /FAN1_PWM
- J13 pad 3: /BrakeADC -> /FAN1_TACH
- J13 pad 4: /Accel_ADC -> /MCU + Peripherals/SDA
- J13 pad 5: /MCU + Peripherals/LDAC -> /MCU + Peripherals/SCL
- J7 pad 1: /Brake_Vref -> Net-(J7-Pin_1)
- J7 pad 10: Net-(J7-Pin_10) -> Net-(J7-Pin_1)
- J7 pad 2: /Accel_Vref -> /Mtr_Pulse
- J7 pad 4: /Mtr_Pulse -> /Accel_Vref
- J7 pad 5: Net-(J7-Pin_5) -> /Brake_Vref
- J7 pad 6: Net-(J7-Pin_5) -> Net-(J7-Pin_6)
- J7 pad 7: GND_ISO -> Net-(J7-Pin_6)
- J7 pad 9: Net-(J7-Pin_10) -> GND_ISO
- J8 pad 1: /Moco_LED+ -> Net-(J8-Pin_1)
- J8 pad 10: /map_bit1_sig -> /FR_MODE_IN
- J8 pad 12: /FR_MODE_IN -> /map_bit1_sig
- J8 pad 13: /PWR_MODE_OUT -> /map_bit3_sig
- J8 pad 14: /Moco_LED- -> Net-(J8-Pin_1)
- J8 pad 2: /PWR_MODE_IN -> /map_bit2_sig
- J8 pad 3: /FR_MODE_OUT -> /map_bit0_sig
- J8 pad 5: /map_bit0_sig -> /FR_MODE_OUT
- J8 pad 6: /map_bit2_sig -> /PWR_MODE_IN
- J8 pad 7: Net-(J8-Pin_7) -> /Moco_LED+
- J8 pad 8: Net-(J8-Pin_7) -> /Moco_LED-
- J8 pad 9: /map_bit3_sig -> /PWR_MODE_OUT
- JP5 pad 1: +3.3V -> +5V
- L2 pad 1: +3.3V -> +5V
- R2 pad 1: Net-(J7-Pin_5) -> Net-(J7-Pin_1)
- R3 pad 1: Net-(J8-Pin_7) -> Net-(J8-Pin_1)
- U2 pad 2: /Power Regulation/LDO/Vin -> +5V
- U2 pad 7: /Power Regulation/LDO/Vin -> +5V
- U4 pad 55: /MCU + Peripherals/100PinMCU/PD8 -> /MCU + Peripherals/ESTOP_Fault
- U4 pad 56: /MCU + Peripherals/100PinMCU/PD9 -> /MCU + Peripherals/SWOC
- U4 pad 88: /MCU + Peripherals/100PinMCU/PD6 -> /MCU + Peripherals/Mtr_Fault
- U4 pad 89: /MCU + Peripherals/100PinMCU/PD7 -> /MCU + Peripherals/BPS_Fault
Routing:
- net Net-(JP1-A): track 14.8 -> 0.00 mm
- net /CarCAN_L: track 10.1 -> 0.00 mm, vias 2 -> 0
- net Net-(J10-Pin_3): track 8.21 -> 0.00 mm
- net /CarCAN_H: track 6.22 -> 0.00 mm, vias 1 -> 0
- net Net-(J10-Pin_4): track 5.77 -> 0.00 mm
- net Net-(C23-Pad2): track 4.04 -> 0.00 mm
- net /Power Regulation/Vout_pp: vias 8 -> 0
Other:
- board text removed: "Galvanic Isolation"
