File: Hardware/VehicleControlUnit/VehicleControlUnit.kicad_pcb (KiCad board)
At the start: 4 copper layers, 100 x 80 mm, 218 parts, among them IC1 LM74502DDFR, IC2 TCAN3413DR, IC3 EMC2305-1-AP-TR, IC4 ISO7741DWR, IC5 ISO7741DWR, IC6 ISO7741DWR, IC7 ISO1042QDWRQ1, J1 CAN_DEBUG_NANO_01x04, J10 SWD_Header, J11 SWD, J12 Micro_SD_Card_Det2, J13 Fan_Debug_Conn, J14 Debug_Conn1, J15 Debug_Conn2, J16 USB_C_Receptacle_USB2.0_16P, J2 WaveSculptor Debug, J3 CAN_NANO_01x03, J4 Thermistor, J5 CAN_NANO_01x03, J6 Fan_Conn1, J7 MotorConn_1, J8 Motor_Conn2, J9 Fan_Conn2, Q1 PSMN012-100YS, Q2 PSMN012-100YS, Q3 IRLML2030TRPBF, Q4 DMP3099L-7, Q5 IRLML2030TRPBF, Q6 IRLML2030TRPBF, Q7 IRLML2030TRPBF, Q8 IRLML2030TRPBF, SW1 SW_SPDT, U1 LMR51635XDDCR, U2 TPS2117DRLR, U3 MCP1826S, U4 STM32G473VETx, U5 MCP4922T-E/ST, Y1 Crystal

Commit message: baboosh
Parts:
- R69: moved to B.Cu
- moved D31 33.1 mm to (146.3, 81.4), turned to 180 degrees
- moved R68 31.0 mm to (146.4, 81.5), turned to 180 degrees
- moved TP3 24.4 mm to (124.0, 85.0), turned to -90 degrees
- moved TP4 23.0 mm to (114.2, 85.0), turned to -90 degrees
- moved TP2 22.7 mm to (119.0, 85.0), turned to -90 degrees
- moved C19 12.9 mm to (139.2, 76.5), turned to -90 degrees
- moved R9 12.7 mm to (126.9, 68.4)
- moved C13 12.5 mm to (113.6, 79.5), turned to 90 degrees
- moved C2 10.6 mm to (137.0, 70.0)
- moved IC1 10.6 mm to (132.7, 68.8)
- moved Q2 10.6 mm to (129.2, 63.9)
- moved D1 10.6 mm to (132.8, 64.2)
- moved R4 10.6 mm to (138.6, 68.5)
- moved C5 10.6 mm to (129.5, 60.8)
- moved C7 10.6 mm to (127.6, 69.1)
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
Commit message: im hungryyyyyyyyyy
Parts:
- moved D8 2.41 mm to (136.3, 82.0)
- moved R24 2.41 mm to (136.3, 81.9)
- moved TP2 0.25 mm to (119.0, 85.2)
- moved TP3 0.25 mm to (124.0, 85.2)
- moved TP4 0.25 mm to (114.2, 85.2)
- moved TP_3.3V1 0.25 mm to (130.0, 85.2)
Changed lines of the file:
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@@
 	(footprint "TestPoint:TestPoint_THTPad_D3.0mm_Drill1.5mm"
 		(layer "F.Cu")
-		(at 119 85 -90)
+		(at 119 85.25 -90)
 		(descr "THT pad as test Point, diameter 3.0mm, hole diameter 1.5mm")
 		(tags "test point THT pad")
@@
 	(footprint "TestPoint:TestPoint_THTPad_D3.0mm_Drill1.5mm"
 		(layer "F.Cu")
-		(at 114.25 85 -90)
+		(at 114.25 85.25 -90)
 		(descr "THT pad as test Point, diameter 3.0mm, hole diameter 1.5mm")
 		(tags "test point THT pad")
@@
 	(footprint "LED_SMD:LED_0603_1608Metric"
 		(layer "F.Cu")
-		(at 138.7 81.95)
+		(at 136.2875 81.95)
 		(descr "LED SMD 0603 (1608 Metric), square (rectangular) end terminal, IPC-7351 nominal, (Body size source: http://www.tortai-tech.com/upload/download/2011102023233369053.pdf)")
 		(tags "LED")
@@
 	(footprint "TestPoint:TestPoint_Loop_D1.80mm_Drill1.0mm_Beaded"
 		(layer "F.Cu")
-		(at 130 85 90)
+		(at 130 85.25 90)
 		(descr "wire loop with bead as test point, loop diameter 1.8mm, hole diameter 1.0mm")
 		(tags "test point wire loop bead")
@@
 	(footprint "TestPoint:TestPoint_THTPad_D3.0mm_Drill1.5mm"
 		(layer "F.Cu")
-		(at 124 85 -90)
+		(at 124 85.25 -90)
 		(descr "THT pad as test Point, diameter 3.0mm, hole diameter 1.5mm")
 		(tags "test point THT pad")
@@
 		(tags "capacitor handsolder")
 		(property "Reference" "C19"
-			(at 6.807482 -0.412084 180)
+			(at 6.807482 2.000416 180)
 			(layer "B.SilkS")
 			(effects
@@
 	(footprint "Resistor_SMD:R_0603_1608Metric_Pad0.98x0.95mm_HandSolder"
 		(layer "B.Cu")
-		(at 138.7425 81.91)
+		(at 136.33 81.91)
 		(descr "Resistor SMD 0603 (1608 Metric), square (rectangular) end terminal, IPC-7351 nominal with elongated pad for handsoldering. (Body size source: IPC-SM-782 page 72, https://www.pcb-3d.com/wordpress/wp-content/uploads/ipc-sm-782a_amendment_1_and_2.pdf)")
 		(tags "resistor handsolder")

Commit message: tracing in progress....
Parts:
- added C41: 0.1u, Capacitor_SMD:C_0603_1608Metric_Pad1.08x0.95mm_HandSolder, B.Cu at (158.7, 80.8)
- added C42: 0.1u, Capacitor_SMD:C_0603_1608Metric_Pad1.08x0.95mm_HandSolder, B.Cu at (158.7, 84.2)
- added C43: 0.1u, Capacitor_SMD:C_0603_1608Metric_Pad1.08x0.95mm_HandSolder, B.Cu at (158.8, 92.1)
- added C44: 0.1u, Capacitor_SMD:C_0603_1608Metric_Pad1.08x0.95mm_HandSolder, B.Cu at (158.8, 95.5)
- added C45: 0.1u, Capacitor_SMD:C_0603_1608Metric_Pad1.08x0.95mm_HandSolder, F.Cu at (158.3, 148.6)
- added C46: 0.1u, Capacitor_SMD:C_0603_1608Metric_Pad1.08x0.95mm_HandSolder, F.Cu at (158.3, 151.1)
- added C47: 0.1u, Capacitor_SMD:C_0603_1608Metric_Pad1.08x0.95mm_HandSolder, F.Cu at (162.6, 138.6)
- added C48: 0.1u, Capacitor_SMD:C_0603_1608Metric_Pad1.08x0.95mm_HandSolder, F.Cu at (162.6, 141.1)
- added C49: 0.1u, Capacitor_SMD:C_0603_1608Metric_Pad1.08x0.95mm_HandSolder, F.Cu at (162.6, 143.6)
- added C50: 0.1u, Capacitor_SMD:C_0603_1608Metric_Pad1.08x0.95mm_HandSolder, F.Cu at (162.6, 146.1)
- added C51: 0.1u, Capacitor_SMD:C_0603_1608Metric_Pad1.08x0.95mm_HandSolder, F.Cu at (162.6, 148.6)
- added C52: 0.1u, Capacitor_SMD:C_0603_1608Metric_Pad1.08x0.95mm_HandSolder, F.Cu at (162.6, 151.1)
- added C56: 0.1u, Capacitor_SMD:C_0603_1608Metric_Pad1.08x0.95mm_HandSolder, F.Cu at (167.0, 138.6)
- added C57: 0.1u, Capacitor_SMD:C_0603_1608Metric_Pad1.08x0.95mm_HandSolder, F.Cu at (167.0, 141.1)
- added C58: 0.1u, Capacitor_SMD:C_0603_1608Metric_Pad1.08x0.95mm_HandSolder, F.Cu at (167.0, 143.6)
- added C59: 0.1u, Capacitor_SMD:C_0603_1608Metric_Pad1.08x0.95mm_HandSolder, F.Cu at (167.0, 146.1)
- moved JP6 21.5 mm to (137.8, 58.2), turned to -90 degrees
- moved R13 11.0 mm to (133.3, 103.6), turned to 90 degrees
- moved D4 10.6 mm to (135.3, 103.4), turned to 90 degrees
- moved R14 10.3 mm to (135.2, 103.6), turned to -90 degrees
- moved C23 10.2 mm to (137.2, 103.6), turned to 90 degrees
- moved C14 6.18 mm to (126.1, 78.2), turned to -90 degrees
- moved JP1 5.77 mm to (139.8, 110.4), turned to 180 degrees
- moved C22 4.36 mm to (133.3, 109.1), turned to 90 degrees
- moved C20 2.88 mm to (136.9, 109.2), turned to -90 degrees
- moved C21 2.85 mm to (134.9, 109.1), turned to 90 degrees
- moved IC2 2.61 mm to (135.2, 109.1), turned to 90 degrees
- moved TP2 1.95 mm to (119.0, 87.2)
- moved TP3 1.95 mm to (124.0, 87.2)
- moved TP4 1.95 mm to (114.2, 87.2)
- moved R43 1.55 mm to (94.9, 75.5)
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- renumbered C42 to C53, C43 to C54, C41 to C55, C44 to C60, C45 to C61, C46 to C62, C47 to C63, C48 to C64, C49 to C65, C50 to C66
Connections:
- net /Power Regulation/PowerProtection/Vin renamed /Power Regulation/Vin_PP
- J13 pad 2: /FAN1_PWM -> /FAN1_TACH
- J13 pad 3: /FAN1_TACH -> /FAN1_PWM
- J6 pad 2: /FAN1_TACH -> /FAN1_PWM
- J6 pad 3: /FAN1_PWM -> /FAN1_TACH
- J9 pad 2: /FAN2_TACH -> /FAN2_PWM
- J9 pad 3: /FAN2_PWM -> /FAN2_TACH
Routing:
- net GND: track 0.00 -> 77.7 mm, vias 0 -> 32
- net +3.3V: track 0.00 -> 52.4 mm, vias 0 -> 8
- net /CarCAN_L: track 0.00 -> 38.6 mm, vias 0 -> 1
- net /Power Regulation/5V_Buck: track 0.00 -> 37.5 mm, vias 0 -> 4
- net /Power Regulation/Vin_PP: track 0.00 -> 37.0 mm, vias 0 -> 8
- net /CarCAN_H: track 0.00 -> 33.7 mm, vias 0 -> 1
- net /FAN1_PWM: track 0.00 -> 32.6 mm, vias 0 -> 2
- net /FAN1_TACH: track 0.00 -> 31.2 mm, vias 0 -> 2
- net /Power Regulation/12VBuck/SW: track 0.00 -> 25.0 mm, vias 0 -> 1
- net /MCU + Peripherals/SCL: track 0.00 -> 25.0 mm
- net /Power Regulation/12VBuck/FB: track 0.00 -> 22.1 mm, vias 0 -> 1
- net /Power Regulation/12VBuck/CB: track 0.00 -> 21.0 mm, vias 0 -> 2
- net /MCU + Peripherals/SDA: track 0.00 -> 19.4 mm
- net /MCU + Peripherals/ALERT: track 0.00 -> 14.7 mm
- net Net-(J3-SHIELD): track 0.00 -> 14.1 mm
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- added copper zone on F.Cu, net +12V
- added copper zone on In2.Cu, net +12V
- added copper zone on F.Cu, net +3.3V
- added copper zone on In2.Cu, net +3.3V
- added copper zone on In2.Cu, net /+12V_PP
- added copper zone on F.Cu, net /Power Regulation/5V_Buck
- added copper zone on B.Cu, net /Power Regulation/Vin_PP
- added copper zone on F.Cu, net /Power Regulation/Vin_PP
- added copper zone on F.Cu, net /Power Regulation/Vout_pp
- added copper zone on In1.Cu, net GND
- added copper zone on In1.Cu, net GND_ISO
