File: Hardware/VehicleControlUnit/VehicleControlUnit.kicad_pcb (KiCad board)
At the start: 4 copper layers, 100 x 80 mm, 240 parts, among them IC1 LM74502DDFR, IC2 TCAN3413DR, IC3 EMC2305-1-AP-TR, IC4 ISO7741DWR, IC5 ISO7741DWR, IC6 ISO7741DWR, IC7 ISO1042QDWRQ1, J1 CAN_DEBUG_NANO_01x04, J11 SWD_Header, J12 SWD, J13 Micro_SD_Card_Det2, J14 Fan_Debug_Conn, J15 PH1, J16 PH2, J17 Debug_Conn2, J18 PH4, J19 PH3, J2 WaveSculptor_CAN, J20 USB_C_Receptacle_USB2.0_16P, J3 WaveSculptor_PWR, J4 CAN_NANO_02x03, J5 Thermistor, J6 Fan_Conn1, J7 MotorConn_1, J8 Motor_Conn2, J9 Fan_Conn2, Q1 PSMN012-100YS, Q2 PSMN012-100YS, Q3 IRLML2030TRPBF, Q4 DMP3099L-7, Q5 IRLML2030TRPBF, Q6 IRLML2030TRPBF, Q7 IRLML2030TRPBF, Q8 IRLML2030TRPBF, SW1 SW_SPDT, U1 LMR51635XDDCR, U2 TPS2117DRLR, U3 MCP1826S, U4 STM32G473VETx, U5 MCP4922T-E/ST, Y1 Crystal

Commit message: dsalkf ljhhk;sdf
Other:
- board text added: "LED+ LED- PM_IN PM_O FR_O FR_IN MB0 MB1 MB2 -V_mtr MB3 +V_mtr --SHLD--"
- board text added: "Mika"
- board text added: "PM_G FRM_G MB1_G MB3_G CLK CS Acc_ADC +ISO MB0_G MB2_G MOSI -ISO -ISO BR_ADC"
- board text removed: "LED+ LED- PM_IN FR_IN PM_O FR_O MB0 MB1 MB2 -Vin MB3 +Vin --SHLD--"
- board text removed: "PM_G FRM_G MB1_G MB3_G CLK CS Acc_ADC +ISO MB0_G MB2_G MOSI -ISO ISO BR_ADC"
Changed lines of the file:
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@@
 		(tags "Integrated Circuit")
 		(property "Reference" "IC4"
-			(at 4.421892 -6.799048 180)
+			(at -4.328108 -6.324048 180)
 			(layer "F.SilkS")
 			(effects
@@
 		(at 158.728108 61.185335)
 		(property "Reference" "L2"
-			(at -0.228108 2.314665 0)
+			(at -2.553108 -0.035335 0)
 			(layer "F.SilkS")
 			(effects
@@
 	)
 	(gr_line
-		(start 175.65 106.625)
-		(end 168.05 106.625)
+		(start 175.6625 113.625)
+		(end 175.6 108.1)
 		(stroke
 			(width 0.1)
@@
 	)
 	(gr_line
-		(start 175.65 106.625)
-		(end 175.65 97.275)
+		(start 175.7 113.65)
+		(end 168.05 113.65)
 		(stroke
 			(width 0.1)
@@
 	)
 	(gr_line
-		(start 175.6625 113.625)
-		(end 175.6 108.1)
+		(start 175.825 96.9)
+		(end 176.75 96.9)
 		(stroke
-			(width 0.1)
-			(type default)
+			(width 0.5)
+			(type solid)
 		)
 		(layer "F.SilkS")
 	)
 	(gr_line
-		(start 175.7 113.65)
-		(end 168.05 113.65)
+		(start 175.925 106.625)
+		(end 168.05 106.625)
 		(stroke
 			(width 0.1)
@@
 	)
 	(gr_line
-		(start 175.825 96.9)
-		(end 176.75 96.9)
+		(start 175.925 106.625)
+		(end 175.925 96.95)
 		(stroke
-			(width 0.5)
-			(type solid)
+			(width 0.1)
+			(type default)
 		)
 		(layer "F.SilkS")
@@
 		)
 	)
+	(gr_text "Mika"
+		(at 163.025 62.575 0)
+		(layer "F.Mask")
+		(effects
+			(font
+				(size 2 2)
+				(thickness 0.3)
+				(bold yes)
+			)
+			(justify left bottom)
+		)
+	)
 	(gr_text "Ac_ADC Pulse\nAcc_V  MCAN_H\nBr_V   MCAN_L\nBr_ADC -ISO\n---SHLD---"
 		(at 168.35 113.275 0)
@@
 	(gr_text "MB3_G"
 		(at 175.038108 85.389048 0)
-		(layer "F.SilkS" knockout)
+		(layer "F.SilkS")
 		(effects
 			(font
@@
 	(gr_text "MB2_G"
 		(at 175.088108 81.789048 0)
-		(layer "F.SilkS" knockout)
+		(layer "F.SilkS")
 		(effects
 			(font
@@
 	(gr_text "MB1_G"
 		(at 175.1 77.8 0)
-		(layer "F.SilkS" knockout)
+		(layer "F.SilkS")
 		(effects
 			(font
@@
 	(gr_text "PM_G"
 		(at 175.15 66.7 0)
-		(layer "F.SilkS" knockout)
+		(layer "F.SilkS")
 		(effects
 			(font
@@
 	(gr_text "FRM_G"
 		(at 175.15 70.7 0)
-		(layer "F.SilkS" knockout)
+		(layer "F.SilkS")
 		(effects
 			(font
@@
 	(gr_text "MB0_G"
 		(at 175.15 74.2 0)
-		(layer "F.SilkS" knockout)
+		(layer "F.SilkS")
 		(effects
 			(font
@@
 		)
 	)
-	(gr_text "MB2"
-		(at 151.4 91.175 0)
-		(layer "F.SilkS" knockout)
+	(gr_text "LDAC"
+		(at 151.325 93.9 0)
+		(layer "F.SilkS")
 		(effects
 			(font
@@
 		)
 	)
-	(gr_text "MB3"
-		(at 151.525 96.35 0)
-		(layer "F.SilkS" knockout)
+	(gr_text "MB2"
+		(at 151.4 91.175 0)
+		(layer "F.SilkS")
 		(effects
 			(font
@@
 		)
 	)
-	(gr_text "LDAC"
-		(at 151.625 93.9 0)
-		(layer "F.SilkS" knockout)
+	(gr_text "MB3"
+		(at 151.525 96.35 0)
+		(layer "F.SilkS")
 		(effects
 			(font
@@
 		)
 	)
-	(gr_text "PM_G FRM_G MB1_G MB3_G CLK CS Acc_ADC\n+ISO MB0_G MB2_G MOSI  -ISO ISO BR_ADC  "
+	(gr_text "PM_G FRM_G MB1_G MB3_G CLK CS Acc_ADC\n+ISO MB0_G MB2_G MOSI -ISO -ISO BR_ADC  "
 		(at 158.2 122.4 0)
 		(layer "F.SilkS" knockout)
@@
 		)
 	)
-	(gr_text "LED+  LED-\nPM_IN FR_IN \nPM_O  FR_O\nMB0   MB1\nMB2   -Vin\nMB3   +Vin\n--SHLD--\n"
+	(gr_text "LED+  LED-\nPM_IN PM_O \nFR_O  FR_IN\nMB0   MB1\nMB2  -V_mtr\nMB3  +V_mtr\n--SHLD--\n"
 		(at 172 106.025 0)
 		(layer "F.SilkS")
