File: Hardware/VehicleControlUnit/12VBuck.kicad_sch (KiCad schematic)
At the start: 14 parts, among them U1 LMR51635XDDCR

Commit message: i hate this moco, its so stupid why are we doign this.
Parts:
- renumbered R11 to R10, R12 to R11
Changed lines of the file:
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@@
 		(dnp no)
 		(fields_autoplaced yes)
-		(property "Reference" "#FLG05"
+		(property "Reference" "#FLG06"
 			(at 149.86 79.375 0)
 			(hide yes)
@@
 			(project "VehicleControlUnit"
 				(path "/e864fac9-3897-46c9-9101-6d5488c6cd3a/f16a8bc3-f058-4d27-badd-0afc148d009e/890fb496-5953-4e5b-b8ad-28917c0a3c13"
-					(reference "#FLG05")
+					(reference "#FLG06")
 					(unit 1)
 				)
@@
 		(dnp no)
 		(fields_autoplaced yes)
-		(property "Reference" "#FLG07"
+		(property "Reference" "#FLG08"
 			(at 179.07 84.455 0)
 			(hide yes)
@@
 			(project "VehicleControlUnit"
 				(path "/e864fac9-3897-46c9-9101-6d5488c6cd3a/f16a8bc3-f058-4d27-badd-0afc148d009e/890fb496-5953-4e5b-b8ad-28917c0a3c13"
-					(reference "#FLG07")
+					(reference "#FLG08")
 					(unit 1)
 				)
@@
 		(dnp no)
 		(fields_autoplaced yes)
-		(property "Reference" "#FLG04"
+		(property "Reference" "#FLG05"
 			(at 88.9 79.375 0)
 			(hide yes)
@@
 			(project "VehicleControlUnit"
 				(path "/e864fac9-3897-46c9-9101-6d5488c6cd3a/f16a8bc3-f058-4d27-badd-0afc148d009e/890fb496-5953-4e5b-b8ad-28917c0a3c13"
-					(reference "#FLG04")
+					(reference "#FLG05")
 					(unit 1)
 				)
@@
 		(in_pos_files yes)
 		(dnp no)
-		(property "Reference" "#FLG06"
+		(property "Reference" "#FLG07"
 			(at 149.86 84.455 0)
 			(hide yes)
@@
 			(project "VehicleControlUnit"
 				(path "/e864fac9-3897-46c9-9101-6d5488c6cd3a/f16a8bc3-f058-4d27-badd-0afc148d009e/890fb496-5953-4e5b-b8ad-28917c0a3c13"
-					(reference "#FLG06")
+					(reference "#FLG07")
 					(unit 1)
 				)
@@
 		(dnp no)
 		(fields_autoplaced yes)
-		(property "Reference" "R11"
+		(property "Reference" "R10"
 			(at 227.33 85.0899 0)
 			(show_name no)
@@
 			(project "VehicleControlUnit"
 				(path "/e864fac9-3897-46c9-9101-6d5488c6cd3a/f16a8bc3-f058-4d27-badd-0afc148d009e/890fb496-5953-4e5b-b8ad-28917c0a3c13"
-					(reference "R11")
+					(reference "R10")
 					(unit 1)
 				)
@@
 		(dnp no)
 		(fields_autoplaced yes)
-		(property "Reference" "R12"
+		(property "Reference" "R11"
 			(at 227.33 92.7099 0)
 			(show_name no)
@@
 			(project "VehicleControlUnit"
 				(path "/e864fac9-3897-46c9-9101-6d5488c6cd3a/f16a8bc3-f058-4d27-badd-0afc148d009e/890fb496-5953-4e5b-b8ad-28917c0a3c13"
-					(reference "R12")
-					(unit 1)
-				)
+					(reference "R11")
+					(unit 1)
+				)

Commit message: 70% tracing done
Parts:
- renumbered R10 to R11, R11 to R12
Changed lines of the file:
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@@
 		(dnp no)
 		(fields_autoplaced yes)
-		(property "Reference" "R10"
+		(property "Reference" "R11"
 			(at 227.33 85.0899 0)
 			(show_name no)
@@
 			(project "VehicleControlUnit"
 				(path "/e864fac9-3897-46c9-9101-6d5488c6cd3a/f16a8bc3-f058-4d27-badd-0afc148d009e/890fb496-5953-4e5b-b8ad-28917c0a3c13"
-					(reference "R10")
+					(reference "R11")
 					(unit 1)
 				)
@@
 		(dnp no)
 		(fields_autoplaced yes)
-		(property "Reference" "R11"
+		(property "Reference" "R12"
 			(at 227.33 92.7099 0)
 			(show_name no)
@@
 			(project "VehicleControlUnit"
 				(path "/e864fac9-3897-46c9-9101-6d5488c6cd3a/f16a8bc3-f058-4d27-badd-0afc148d009e/890fb496-5953-4e5b-b8ad-28917c0a3c13"
-					(reference "R11")
-					(unit 1)
-				)
+					(reference "R12")
+					(unit 1)
+				)
