File: Hardware/VehicleControlUnit/MUC_Peripherals.kicad_sch (KiCad schematic)
At the start: 15 parts

Commit message: mikas paradise
Parts:
- added D? (x2): LED, LED_SMD:LED_0603_1608Metric, symbol Device:LED
- added R? (x2): 120, Resistor_SMD:R_0603_1608Metric_Pad0.98x0.95mm_HandSolder, symbol Device:R
Connections:
- new net: D?.1 (K), R?.1 (x2)
- new net SW_LED3: D?.2 (A)
- new net SW_LED4: D?.2 (A)
- no-connect marks 50 -> 49
Other:
- moved on the sheet: D10, D11, D12, D13, D14, D8, D9, R25, R26, R27, R28, R29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

Commit message: i hate this moco, its so stupid why are we doign this.
Parts:
- added C38: 1uF, Capacitor_SMD:C_0603_1608Metric_Pad1.08x0.95mm_HandSolder, symbol Device:C
- gave numbers to parts that had none: 4
- renumbered R24 to R23, R25 to R24, R26 to R25, R27 to R26, R28 to R27, R29 to R28, R30 to R29, R31 to R30
Connections:
- net ADC2_IN6+: now also C38.2
- net ADC2_IN6-: now also R31.2, R32.2, C38.1

Commit message: put puzzle togaehtrwetr
Connections:
- net ADC2_IN6+ renamed +TH
- net ADC2_IN6- renamed -TH
Changed lines of the file:
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@@
 	)
 	(junction
-		(at 114.935 38.1)
+		(at 100.33 27.94)
 		(diameter 0)
 		(color 0 0 0 0)
 	)
 	(junction
-		(at 100.33 27.94)
+		(at 114.935 38.1)
 		(diameter 0)
 		(color 0 0 0 0)
@@
 	(wire
 		(pts
-			(xy 114.935 38.1) (xy 116.84 38.1)
+			(xy 114.935 38.1) (xy 123.19 38.1)
 		)
 		(stroke
@@
 		)
 	)
+	(hierarchical_label "-TH"
+		(shape input)
+		(at 100.33 34.29 0)
+		(effects
+			(font
+				(size 1.27 1.27)
+			)
+			(justify left)
+		)
+	)
 	(hierarchical_label "{DAC_SPI}"
 		(shape bidirectional)
@@
 	(hierarchical_label "GND"
 		(shape input)
-		(at 116.84 38.1 0)
+		(at 123.19 38.1 0)
 		(effects
 			(font
@@
 		)
 	)
-	(hierarchical_label "ADC2_IN6+"
+	(hierarchical_label "+TH"
 		(shape input)
 		(at 116.84 27.94 0)
@@
 		)
 	)
-	(hierarchical_label "ADC2_IN6-"
-		(shape input)
-		(at 100.33 34.29 0)
-		(effects
-			(font
-				(size 1.27 1.27)
-			)
-			(justify left)
-		)
-	)
 	(hierarchical_label "PWR_EN"
 		(shape output)
@@
 		(dnp no)
 		(property "Reference" "C38"
-			(at 113.665 30.48 0)
+			(at 111.76 29.21 0)
 			(show_name no)
 			(do_not_autoplace no)

Commit message: layoutttttttttttttttttttttttttttttttttttt
Parts:
- added D13, D14, D15, D16, D17: LED, LED_SMD:LED_0603_1608Metric, symbol Device:LED
- added R33, R34, R35, R36, R37: 250, Resistor_SMD:R_0603_1608Metric_Pad0.98x0.95mm_HandSolder, symbol Device:R
- R24, R26, R27, R28, R29, R30, R31, R32: value 120 -> 250
- renumbered D13 to D18, D14 to D19, D15 to D20, D16 to D21
Connections:
- net -TH: now also R33.2, R34.2, R35.2, R36.2, R37.2
- net at R30.1: now also D14.1 (K); no longer D19.1 (K)
- net at R32.1: now also D16.1 (K); no longer D21.1 (K)
- net at D18.1 (K): now also R34.1; no longer R29.1
- net at D20.1 (K): now also R36.1; no longer R31.1
- new net: D19.1 (K), R35.1
- new net: D13.1 (K), R29.1
- new net: D17.1 (K), R33.1
- new net: D15.1 (K), R31.1
- new net: D21.1 (K), R37.1
- new net BPS_Fault: D15.2 (A)
- new net ESTOP_Fault: D16.2 (A)
- new net HB_LED: D13.2 (A)
- new net Mtr_Fault: D14.2 (A)
- new net SWOC: D17.2 (A)
Other:
- moved on the sheet: C38, D10, D11, D12, D18, D19, D20, D21, D8, D9, R23, R24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

Commit message: migtve finally lcokeefd in = ggs
Connections:
- no-connect marks 49 -> 45
Changed lines of the file:
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@@
 	)
 	(no_connect
-		(at 82.55 99.06)
-	)
-	(no_connect
 		(at 40.64 116.84)
 	)
@@
 	)
 	(no_connect
-		(at 82.55 96.52)
-	)
-	(no_connect
 		(at 40.64 88.9)
 	)
@@
 	)
 	(no_connect
-		(at 82.55 93.98)
-	)
-	(no_connect
 		(at 82.55 133.35)
 	)
@@
 	)
 	(no_connect
-		(at 82.55 91.44)
-	)
-	(no_connect
 		(at 40.64 134.62)
 	)
@@
 	(wire
 		(pts
-			(xy 81.28 91.44) (xy 82.55 91.44)
+			(xy 81.28 91.44) (xy 85.09 91.44)
 		)
 		(stroke
@@
 	(wire
 		(pts
-			(xy 81.28 93.98) (xy 82.55 93.98)
+			(xy 81.28 93.98) (xy 85.09 93.98)
 		)
 		(stroke
@@
 	(wire
 		(pts
-			(xy 81.28 99.06) (xy 82.55 99.06)
+			(xy 81.28 99.06) (xy 85.09 99.06)
 		)
 		(stroke
@@
 	(wire
 		(pts
-			(xy 81.28 96.52) (xy 82.55 96.52)
+			(xy 81.28 96.52) (xy 85.09 96.52)
 		)
 		(stroke
@@
 		)
 	)
+	(label "SWOC"
+		(at 85.09 99.06 0)
+		(effects
+			(font
+				(size 1.27 1.27)
+			)
+			(justify left bottom)
+		)
+	)
+	(label "BPS_Fault"
+		(at 85.09 93.98 0)
+		(effects
+			(font
+				(size 1.27 1.27)
+			)
+			(justify left bottom)
+		)
+	)
 	(label "SW_LED3"
 		(at 85.09 83.82 0)
@@
 		)
 	)
+	(label "Mtr_Fault"
+		(at 85.09 91.44 0)
+		(effects
+			(font
+				(size 1.27 1.27)
+			)
+			(justify left bottom)
+		)
+	)
 	(label "CLK"
 		(at 87.63 58.42 180)
@@
 		)
 	)
+	(label "ESTOP_Fault"
+		(at 85.09 96.52 0)
+		(effects
+			(font
+				(size 1.27 1.27)
+			)
+			(justify left bottom)
+		)
+	)

Commit message: 70% tracing done
Parts:
- renumbered R23 to R24, R24 to R25, R25 to R26, R26 to R27, R27 to R28, R28 to R29, R29 to R30, R30 to R31, R31 to R32, R32 to R33, R33 to R34, R34 to R35, R35 to R36, R36 to R37, R37 to R38
Connections:
- no-connect marks 45 -> 43
