File: Hardware/VehicleControlUnit/Power_Regulation.kicad_sch (KiCad schematic)
At the start: 7 parts

Commit message: mika review last time pelase
Other:
- note removed: "Check for power test points"
Changed lines of the file:
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@@
-		)
-	)
-	(text "Check for power test points"
-		(exclude_from_sim no)
-		(at 60.96 84.455 0)
-		(effects
-			(font
-				(size 2.54 2.54)
-				(thickness 0.508)
-				(bold yes)
-			)
 		)
 	)

Commit message: surabhi review pls
Parts:
- renumbered R70 to R74, R71 to R75, R72 to R76
Changed lines of the file:
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@@
 		(in_pos_files yes)
 		(dnp no)
-		(property "Reference" "R70"
+		(property "Reference" "R74"
 			(at 42.418 67.31 90)
 			(show_name no)
@@
 			(project "VehicleControlUnit"
 				(path "/e864fac9-3897-46c9-9101-6d5488c6cd3a/f16a8bc3-f058-4d27-badd-0afc148d009e"
-					(reference "R70")
+					(reference "R74")
 					(unit 1)
 				)
@@
 		(in_pos_files yes)
 		(dnp no)
-		(property "Reference" "R72"
+		(property "Reference" "R76"
 			(at 101.6 68.834 90)
 			(show_name no)
@@
 			(project "VehicleControlUnit"
 				(path "/e864fac9-3897-46c9-9101-6d5488c6cd3a/f16a8bc3-f058-4d27-badd-0afc148d009e"
-					(reference "R72")
+					(reference "R76")
 					(unit 1)
 				)
@@
 		(in_pos_files yes)
 		(dnp no)
-		(property "Reference" "R71"
+		(property "Reference" "R75"
 			(at 101.854 61.976 90)
 			(show_name no)
@@
 			(project "VehicleControlUnit"
 				(path "/e864fac9-3897-46c9-9101-6d5488c6cd3a/f16a8bc3-f058-4d27-badd-0afc148d009e"
-					(reference "R71")
-					(unit 1)
-				)
+					(reference "R75")
+					(unit 1)
+				)
