File: Hardware/VehicleControlUnit/100PinMCU.kicad_sch (KiCad schematic)
At the start: 33 parts, among them J10 SWD_Header, J11 SWD, SW1 SW_SPDT, U4 STM32G473VETx, Y1 Crystal

Commit message: i thuink i finasldlh did vcu and no can mdvoe over to disng miak 2.0w
Connections:
- net OSC_N: now reaches C24.2, U4.12 (PF0-OSC_IN), Y1.2
- net OSC_P: now reaches C25.2, U4.13 (PF1-OSC_OUT), Y1.1
Changed lines of the file:
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@@
+		)
+	)
+	(label "OSC_N"
+		(at 48.26 50.8 0)
+		(effects
+			(font
+				(size 1.27 1.27)
+			)
+			(justify left bottom)
+		)
+	)
+	(label "OSC_P"
+		(at 48.26 58.42 0)
+		(effects
+			(font
+				(size 1.27 1.27)
+			)
+			(justify left bottom)
 		)
 	)
