File: Hardware/VehicleControlUnit/motor_fans.kicad_sch (KiCad schematic)
At the start: 17 parts, among them IC3 EMC2305-1-AP-TR

Commit message: i hate this moco, its so stupid why are we doign this.
Parts:
- renumbered C38 to C39, C39 to C40, D15 to D17, D16 to D18, R34 to R35, R35 to R36, R36 to R37, R37 to R38, R38 to R39, R39 to R40, R40 to R41
Changed lines of the file:
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@@
 		(in_pos_files yes)
 		(dnp no)
-		(property "Reference" "R34"
+		(property "Reference" "R35"
 			(at 62.992 43.18 0)
 			(show_name no)
@@
 			(project "VehicleControlUnit"
 				(path "/e864fac9-3897-46c9-9101-6d5488c6cd3a/76867641-26a4-43d1-a64a-9a6eb791f3f7"
-					(reference "R34")
+					(reference "R35")
 					(unit 1)
 				)
@@
 		(in_pos_files yes)
 		(dnp no)
-		(property "Reference" "R39"
+		(property "Reference" "R40"
 			(at 110.49 43.434 90)
 			(show_name no)
@@
 			(project "VehicleControlUnit"
 				(path "/e864fac9-3897-46c9-9101-6d5488c6cd3a/76867641-26a4-43d1-a64a-9a6eb791f3f7"
-					(reference "R39")
+					(reference "R40")
 					(unit 1)
 				)
@@
 		(in_pos_files yes)
 		(dnp no)
-		(property "Reference" "D16"
+		(property "Reference" "D18"
 			(at 62.484 83.312 0)
 			(show_name no)
@@
 			(project "VehicleControlUnit"
 				(path "/e864fac9-3897-46c9-9101-6d5488c6cd3a/76867641-26a4-43d1-a64a-9a6eb791f3f7"
-					(reference "D16")
+					(reference "D18")
 					(unit 1)
 				)
@@
 		(in_pos_files yes)
 		(dnp no)
-		(property "Reference" "C39"
+		(property "Reference" "C40"
 			(at 57.912 57.15 0)
 			(show_name no)
@@
 			(project "VehicleControlUnit"
 				(path "/e864fac9-3897-46c9-9101-6d5488c6cd3a/76867641-26a4-43d1-a64a-9a6eb791f3f7"
-					(reference "C39")
+					(reference "C40")
 					(unit 1)
 				)
@@
 		(in_pos_files yes)
 		(dnp no)
-		(property "Reference" "R38"
+		(property "Reference" "R39"
 			(at 104.648 81.026 90)
 			(show_name no)
@@
 			(project "VehicleControlUnit"
 				(path "/e864fac9-3897-46c9-9101-6d5488c6cd3a/76867641-26a4-43d1-a64a-9a6eb791f3f7"
-					(reference "R38")
+					(reference "R39")
 					(unit 1)
 				)
@@
 		(in_pos_files yes)
 		(dnp no)
-		(property "Reference" "R40"
+		(property "Reference" "R41"
 			(at 119.888 43.434 90)
 			(show_name no)
@@
 			(project "VehicleControlUnit"
 				(path "/e864fac9-3897-46c9-9101-6d5488c6cd3a/76867641-26a4-43d1-a64a-9a6eb791f3f7"
-					(reference "R40")
+					(reference "R41")
 					(unit 1)
 				)
@@
 		(in_pos_files yes)
 		(dnp no)
-		(property "Reference" "R35"
+		(property "Reference" "R36"
 			(at 68.58 43.18 90)
 			(show_name no)
@@
 			(project "VehicleControlUnit"
 				(path "/e864fac9-3897-46c9-9101-6d5488c6cd3a/76867641-26a4-43d1-a64a-9a6eb791f3f7"
-					(reference "R35")
+					(reference "R36")
 					(unit 1)
 				)
@@
 		(in_pos_files yes)
 		(dnp no)
-		(property "Reference" "C38"
+		(property "Reference" "C39"
 			(at 46.99 57.15 0)
 			(show_name no)
@@
 			(project "VehicleControlUnit"
 				(path "/e864fac9-3897-46c9-9101-6d5488c6cd3a/76867641-26a4-43d1-a64a-9a6eb791f3f7"
-					(reference "C38")
+					(reference "C39")
 					(unit 1)
 				)
@@
 		(in_pos_files yes)
 		(dnp no)
-		(property "Reference" "R37"
+		(property "Reference" "R38"
 			(at 104.14 74.168 90)
 			(show_name no)
@@
 			(project "VehicleControlUnit"
 				(path "/e864fac9-3897-46c9-9101-6d5488c6cd3a/76867641-26a4-43d1-a64a-9a6eb791f3f7"
-					(reference "R37")
+					(reference "R38")
 					(unit 1)
 				)
@@
 		(in_pos_files yes)
 		(dnp no)
-		(property "Reference" "R36"
+		(property "Reference" "R37"
 			(at 77.724 42.672 0)
 			(show_name no)
@@
 			(project "VehicleControlUnit"
 				(path "/e864fac9-3897-46c9-9101-6d5488c6cd3a/76867641-26a4-43d1-a64a-9a6eb791f3f7"
-					(reference "R36")
+					(reference "R37")
 					(unit 1)
 				)
@@
 		(in_pos_files yes)
 		(dnp no)
-		(property "Reference" "D15"
+		(property "Reference" "D17"
 			(at 62.484 73.152 0)
 			(show_name no)
@@
 			(project "VehicleControlUnit"
 				(path "/e864fac9-3897-46c9-9101-6d5488c6cd3a/76867641-26a4-43d1-a64a-9a6eb791f3f7"
-					(reference "D15")
-					(unit 1)
-				)
+					(reference "D17")
+					(unit 1)
+				)

Commit message: layoutttttttttttttttttttttttttttttttttttt
Parts:
- renumbered D17 to D22, D18 to D23, R35 to R40, R36 to R41, R37 to R42, R38 to R43, R39 to R44, R40 to R45, R41 to R46
Other:
- note added: "Fan 1 Flyback"
- note added: "Fan 2 Flyback"
Changed lines of the file:
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@@
 		)
 	)
+	(text "Fan 1 Flyback"
+		(exclude_from_sim no)
+		(at 53.34 74.93 0)
+		(effects
+			(font
+				(size 1.27 1.27)
+			)
+		)
+	)
 	(text "Fan PWM pins configed\nas open drain"
 		(exclude_from_sim no)
@@
 		)
 	)
+	(text "Fan 2 Flyback"
+		(exclude_from_sim no)
+		(at 53.34 88.9 0)
+		(effects
+			(font
+				(size 1.27 1.27)
+			)
+		)
+	)
 	(text "Flyback Diodes"
 		(exclude_from_sim no)
@@
 		(in_pos_files yes)
 		(dnp no)
-		(property "Reference" "R35"
+		(property "Reference" "R40"
 			(at 62.992 43.18 0)
 			(show_name no)
@@
 			(project "VehicleControlUnit"
 				(path "/e864fac9-3897-46c9-9101-6d5488c6cd3a/76867641-26a4-43d1-a64a-9a6eb791f3f7"
-					(reference "R35")
+					(reference "R40")
 					(unit 1)
 				)
@@
 		(in_pos_files yes)
 		(dnp no)
-		(property "Reference" "R40"
+		(property "Reference" "R45"
 			(at 110.49 43.434 90)
 			(show_name no)
@@
 			(project "VehicleControlUnit"
 				(path "/e864fac9-3897-46c9-9101-6d5488c6cd3a/76867641-26a4-43d1-a64a-9a6eb791f3f7"
-					(reference "R40")
+					(reference "R45")
 					(unit 1)
 				)
@@
 		(in_pos_files yes)
 		(dnp no)
-		(property "Reference" "D18"
+		(property "Reference" "D23"
 			(at 62.484 83.312 0)
 			(show_name no)
@@
 		)
 		(property "Value" "D_Schottky"
-			(at 58.42 89.408 0)
+			(at 63.5 88.9 0)
 			(show_name no)
 			(do_not_autoplace no)
@@
 			(project "VehicleControlUnit"
 				(path "/e864fac9-3897-46c9-9101-6d5488c6cd3a/76867641-26a4-43d1-a64a-9a6eb791f3f7"
-					(reference "D18")
+					(reference "D23")
 					(unit 1)
 				)
@@
 		(in_pos_files yes)
 		(dnp no)
-		(property "Reference" "R39"
+		(property "Reference" "R44"
 			(at 104.648 81.026 90)
 			(show_name no)
@@
 			(project "VehicleControlUnit"
 				(path "/e864fac9-3897-46c9-9101-6d5488c6cd3a/76867641-26a4-43d1-a64a-9a6eb791f3f7"
-					(reference "R39")
+					(reference "R44")
 					(unit 1)
 				)
@@
 		(in_pos_files yes)
 		(dnp no)
-		(property "Reference" "R41"
+		(property "Reference" "R46"
 			(at 119.888 43.434 90)
 			(show_name no)
@@
 			(project "VehicleControlUnit"
 				(path "/e864fac9-3897-46c9-9101-6d5488c6cd3a/76867641-26a4-43d1-a64a-9a6eb791f3f7"
-					(reference "R41")
+					(reference "R46")
 					(unit 1)
 				)
@@
 		(in_pos_files yes)
 		(dnp no)
-		(property "Reference" "R36"
+		(property "Reference" "R41"
 			(at 68.58 43.18 90)
 			(show_name no)
@@
 			(project "VehicleControlUnit"
 				(path "/e864fac9-3897-46c9-9101-6d5488c6cd3a/76867641-26a4-43d1-a64a-9a6eb791f3f7"
-					(reference "R36")
+					(reference "R41")
 					(unit 1)
 				)
@@
 		(in_pos_files yes)
 		(dnp no)
-		(property "Reference" "R38"
+		(property "Reference" "R43"
 			(at 104.14 74.168 90)
 			(show_name no)
@@
 			(project "VehicleControlUnit"
 				(path "/e864fac9-3897-46c9-9101-6d5488c6cd3a/76867641-26a4-43d1-a64a-9a6eb791f3f7"
-					(reference "R38")
+					(reference "R43")
 					(unit 1)
 				)
@@
 		(in_pos_files yes)
 		(dnp no)
-		(property "Reference" "R37"
+		(property "Reference" "R42"
 			(at 77.724 42.672 0)
 			(show_name no)
@@
 			(project "VehicleControlUnit"
 				(path "/e864fac9-3897-46c9-9101-6d5488c6cd3a/76867641-26a4-43d1-a64a-9a6eb791f3f7"
-					(reference "R37")
+					(reference "R42")
 					(unit 1)
 				)
@@
 		(in_pos_files yes)
 		(dnp no)
-		(property "Reference" "D17"
+		(property "Reference" "D22"
 			(at 62.484 73.152 0)
 			(show_name no)
@@
 			(project "VehicleControlUnit"
 				(path "/e864fac9-3897-46c9-9101-6d5488c6cd3a/76867641-26a4-43d1-a64a-9a6eb791f3f7"
-					(reference "D17")
+					(reference "D22")
 					(unit 1)
 				)

Commit message: migtve finally lcokeefd in = ggs
Parts:
- removed TP5, TP6, TP7, TP8, TP9: TestPoint, diddle_shah:TestPoint_HEX_3mmID, symbol Connector:TestPoint
- added J13: Fan_Debug_Conn, Connector_PinHeader_2.54mm:PinHeader_1x05_P2.54mm_Vertical, symbol Connector_Generic:Conn_01x05
Connections:
- net ALERT: now also J13.1 (Pin_1)
- net FAN1_PWM: now also J13.2 (Pin_2)
- net FAN1_TACH: now also J13.3 (Pin_3)
- net FAN_SCL: now also J13.5 (Pin_5)
- net FAN_SDA: now also J13.4 (Pin_4)

Commit message: tracing in progress....
Connections:
- net FAN1_PWM: now also J13.3 (Pin_3); no longer J13.2 (Pin_2)
- net FAN1_TACH: now also J13.2 (Pin_2); no longer J13.3 (Pin_3)
Changed lines of the file:
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@@
 	(hierarchical_label "FAN1_PWM"
 		(shape output)
-		(at 151.13 78.105 180)
+		(at 151.13 80.645 180)
 		(effects
 			(font
@@
 	(hierarchical_label "FAN1_TACH"
 		(shape input)
-		(at 151.13 80.645 180)
+		(at 151.13 78.105 180)
 		(effects
 			(font

Commit message: 70% tracing done
Parts:
- renumbered R40 to R41, R41 to R42, R42 to R43, R43 to R44, R44 to R45, R45 to R46, R46 to R47
Changed lines of the file:
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@@
 		(in_pos_files yes)
 		(dnp no)
-		(property "Reference" "R40"
+		(property "Reference" "R41"
 			(at 62.992 43.18 0)
 			(show_name no)
@@
 			(project "VehicleControlUnit"
 				(path "/e864fac9-3897-46c9-9101-6d5488c6cd3a/76867641-26a4-43d1-a64a-9a6eb791f3f7"
-					(reference "R40")
+					(reference "R41")
 					(unit 1)
 				)
@@
 		(in_pos_files yes)
 		(dnp no)
-		(property "Reference" "R45"
+		(property "Reference" "R46"
 			(at 110.49 43.434 90)
 			(show_name no)
@@
 			(project "VehicleControlUnit"
 				(path "/e864fac9-3897-46c9-9101-6d5488c6cd3a/76867641-26a4-43d1-a64a-9a6eb791f3f7"
-					(reference "R45")
+					(reference "R46")
 					(unit 1)
 				)
@@
 		(in_pos_files yes)
 		(dnp no)
-		(property "Reference" "R44"
+		(property "Reference" "R45"
 			(at 104.648 81.026 90)
 			(show_name no)
@@
 			(project "VehicleControlUnit"
 				(path "/e864fac9-3897-46c9-9101-6d5488c6cd3a/76867641-26a4-43d1-a64a-9a6eb791f3f7"
-					(reference "R44")
+					(reference "R45")
 					(unit 1)
 				)
@@
 		(in_pos_files yes)
 		(dnp no)
-		(property "Reference" "R46"
+		(property "Reference" "R47"
 			(at 119.888 43.434 90)
 			(show_name no)
@@
 			(project "VehicleControlUnit"
 				(path "/e864fac9-3897-46c9-9101-6d5488c6cd3a/76867641-26a4-43d1-a64a-9a6eb791f3f7"
-					(reference "R46")
+					(reference "R47")
 					(unit 1)
 				)
@@
 		(in_pos_files yes)
 		(dnp no)
-		(property "Reference" "R41"
+		(property "Reference" "R42"
 			(at 68.58 43.18 90)
 			(show_name no)
@@
 			(project "VehicleControlUnit"
 				(path "/e864fac9-3897-46c9-9101-6d5488c6cd3a/76867641-26a4-43d1-a64a-9a6eb791f3f7"
-					(reference "R41")
+					(reference "R42")
 					(unit 1)
 				)
@@
 		(in_pos_files yes)
 		(dnp no)
-		(property "Reference" "R43"
+		(property "Reference" "R44"
 			(at 104.14 74.168 90)
 			(show_name no)
@@
 			(project "VehicleControlUnit"
 				(path "/e864fac9-3897-46c9-9101-6d5488c6cd3a/76867641-26a4-43d1-a64a-9a6eb791f3f7"
-					(reference "R43")
+					(reference "R44")
 					(unit 1)
 				)
@@
 		(in_pos_files yes)
 		(dnp no)
-		(property "Reference" "R42"
+		(property "Reference" "R43"
 			(at 77.724 42.672 0)
 			(show_name no)
@@
 			(project "VehicleControlUnit"
 				(path "/e864fac9-3897-46c9-9101-6d5488c6cd3a/76867641-26a4-43d1-a64a-9a6eb791f3f7"
-					(reference "R42")
-					(unit 1)
-				)
+					(reference "R43")
+					(unit 1)
+				)

Commit message: DONEEE - silkscreen time
Parts:
- renumbered C39 to C40, C40 to C41, R41 to R42, R42 to R43, R43 to R44, R44 to R45, R45 to R46, R46 to R47, R47 to R48
Changed lines of the file:
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@@
 		(in_pos_files yes)
 		(dnp no)
-		(property "Reference" "R41"
+		(property "Reference" "R42"
 			(at 62.992 43.18 0)
 			(show_name no)
@@
 			(project "VehicleControlUnit"
 				(path "/e864fac9-3897-46c9-9101-6d5488c6cd3a/76867641-26a4-43d1-a64a-9a6eb791f3f7"
-					(reference "R41")
+					(reference "R42")
 					(unit 1)
 				)
@@
 		(in_pos_files yes)
 		(dnp no)
-		(property "Reference" "R46"
+		(property "Reference" "R47"
 			(at 110.49 43.434 90)
 			(show_name no)
@@
 			(project "VehicleControlUnit"
 				(path "/e864fac9-3897-46c9-9101-6d5488c6cd3a/76867641-26a4-43d1-a64a-9a6eb791f3f7"
-					(reference "R46")
+					(reference "R47")
 					(unit 1)
 				)
@@
 		(in_pos_files yes)
 		(dnp no)
-		(property "Reference" "C40"
+		(property "Reference" "C41"
 			(at 57.912 57.15 0)
 			(show_name no)
@@
 			(project "VehicleControlUnit"
 				(path "/e864fac9-3897-46c9-9101-6d5488c6cd3a/76867641-26a4-43d1-a64a-9a6eb791f3f7"
-					(reference "C40")
+					(reference "C41")
 					(unit 1)
 				)
@@
 		(in_pos_files yes)
 		(dnp no)
-		(property "Reference" "R45"
+		(property "Reference" "R46"
 			(at 104.648 81.026 90)
 			(show_name no)
@@
 			(project "VehicleControlUnit"
 				(path "/e864fac9-3897-46c9-9101-6d5488c6cd3a/76867641-26a4-43d1-a64a-9a6eb791f3f7"
-					(reference "R45")
+					(reference "R46")
 					(unit 1)
 				)
@@
 		(in_pos_files yes)
 		(dnp no)
-		(property "Reference" "R47"
+		(property "Reference" "R48"
 			(at 119.888 43.434 90)
 			(show_name no)
@@
 			(project "VehicleControlUnit"
 				(path "/e864fac9-3897-46c9-9101-6d5488c6cd3a/76867641-26a4-43d1-a64a-9a6eb791f3f7"
-					(reference "R47")
+					(reference "R48")
 					(unit 1)
 				)
@@
 		(in_pos_files yes)
 		(dnp no)
-		(property "Reference" "R42"
+		(property "Reference" "R43"
 			(at 68.58 43.18 90)
 			(show_name no)
@@
 			(project "VehicleControlUnit"
 				(path "/e864fac9-3897-46c9-9101-6d5488c6cd3a/76867641-26a4-43d1-a64a-9a6eb791f3f7"
-					(reference "R42")
+					(reference "R43")
 					(unit 1)
 				)
@@
 		(in_pos_files yes)
 		(dnp no)
-		(property "Reference" "C39"
+		(property "Reference" "C40"
 			(at 46.99 57.15 0)
 			(show_name no)
@@
 			(project "VehicleControlUnit"
 				(path "/e864fac9-3897-46c9-9101-6d5488c6cd3a/76867641-26a4-43d1-a64a-9a6eb791f3f7"
-					(reference "C39")
+					(reference "C40")
 					(unit 1)
 				)
@@
 		(in_pos_files yes)
 		(dnp no)
-		(property "Reference" "R44"
+		(property "Reference" "R45"
 			(at 104.14 74.168 90)
 			(show_name no)
@@
 			(project "VehicleControlUnit"
 				(path "/e864fac9-3897-46c9-9101-6d5488c6cd3a/76867641-26a4-43d1-a64a-9a6eb791f3f7"
-					(reference "R44")
+					(reference "R45")
 					(unit 1)
 				)
@@
 		(in_pos_files yes)
 		(dnp no)
-		(property "Reference" "R43"
+		(property "Reference" "R44"
 			(at 77.724 42.672 0)
 			(show_name no)
@@
 			(project "VehicleControlUnit"
 				(path "/e864fac9-3897-46c9-9101-6d5488c6cd3a/76867641-26a4-43d1-a64a-9a6eb791f3f7"
-					(reference "R43")
-					(unit 1)
-				)
+					(reference "R44")
+					(unit 1)
+				)

Commit message: VCU hardware prod files done night night
Parts:
- renumbered J13 to J14
Changed lines of the file:
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@@
 		(in_pos_files yes)
 		(dnp no)
-		(property "Reference" "J13"
+		(property "Reference" "J14"
 			(at 155.575 72.39 0)
 			(show_name no)
@@
 			(project "VehicleControlUnit"
 				(path "/e864fac9-3897-46c9-9101-6d5488c6cd3a/76867641-26a4-43d1-a64a-9a6eb791f3f7"
-					(reference "J13")
+					(reference "J14")
 					(unit 1)
 				)

Commit message: surabhi review pls
Parts:
- renumbered J14 to J13
Changed lines of the file:
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@@
 		(in_pos_files yes)
 		(dnp no)
-		(property "Reference" "J14"
+		(property "Reference" "J13"
 			(at 155.575 72.39 0)
 			(show_name no)
@@
 			(project "VehicleControlUnit"
 				(path "/e864fac9-3897-46c9-9101-6d5488c6cd3a/76867641-26a4-43d1-a64a-9a6eb791f3f7"
-					(reference "J14")
+					(reference "J13")
 					(unit 1)
 				)
